File: Hardware/PCB/sidekickvco/sidekickvco_main.kicad_sch (KiCad schematic)
At the start: 70 parts, among them U1 TL074, U2 TL072, U3 AS3340A, U4 LM4040BIZ-5, U5 LM4040BIZ-5, U6 L79L05_TO92, U8 TL072, U9 TL072

Commit message: Initial version of circuit and layout
Parts:
- removed B1: Board, ao_tht:Board_Marker, symbol ao_symbols:Board
- removed C4, C5: 100nF, ao_tht:C_Disc_D3.0mm_W1.6mm_P2.50mm, symbol ao_symbols:C
- removed GRAF1: Holes, herovco:herovco_panel_behind, symbol ao_symbols:Graphic
- removed H1, H2, H3: MountingHole, ao_tht:MountingHole_3.2mm_M3, symbol ao_symbols:MountingHole
- removed R12, R21: 10k, ao_tht:R_Axial_DIN0207_L6.3mm_D2.5mm_P10.16mm_Horizontal, symbol ao_symbols:R
- removed RV1: 100k, ao_tht:Potentiometer_Alpha_RD901F-40-00D_Single_Vertical_centered, symbol ao_symbols:R_POT
- removed TP1: +12V, ao_tht:TestPoint_THTPad_D1.5mm_Drill0.7mm, symbol Connector:TestPoint
- removed TP3: -12V, ao_tht:TestPoint_THTPad_D1.5mm_Drill0.7mm, symbol Connector:TestPoint
- removed TP5: GND, ao_tht:TestPoint_THTPad_D1.5mm_Drill0.7mm, symbol Connector:TestPoint
- removed U1: TL074, ao_tht:DIP-14_W7.62mm_Socket_LongPads, symbol ao_symbols:TL074
- removed U8, U9: TL072, ao_tht:DIP-8_W7.62mm_Socket_LongPads, symbol ao_symbols:TL072
- added C20: 10nF, ao_tht:C_Rect_L7.2mm_W2.5mm_P5.00mm_FKS2_FKP2_MKS2_MKP2, symbol ao_symbols:C
- added unit 2 of U1
- R10: value 100k -> 1M
- renumbered U2 to U1
Connections:
- net LIN_FM: now also R10.1
- net OCTAVE: now also U1.5 (+)
- net at R4.2: now also U1.6 (-), U1.7
- net at C10.2: now also R8.1
- new net: C20.1, R10.2
- new net: C20.2, R9.1
Other:
- note added: "-5V REGULATOR"
- note added: "Does this work? Or do the CVs need to be summed outside the 3340?"
- note removed: "-5V reg"
- note removed: "POWER CONNECTIONS"
- moved on the sheet: C10, C13, D2, R18, R19, R20, R27, R31, R4, R5, R6, R7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

Commit message: Revise layout, add notes, BUILD.md
Parts:
- RV2: footprint ao_tht:Potentiometer_Bourns_3296W_Vertical_screw_centered -> Potentiometer_THT:Potentiometer_Bourns_3296P_Horizontal
- RV5, RV6: value 20k -> 10k; footprint ao_tht:Potentiometer_Bourns_3296W_Vertical_screw_centered -> Potentiometer_THT:Potentiometer_Bourns_3296P_Horizontal
- RV9: value 50k -> 10k; footprint ao_tht:Potentiometer_Bourns_3296W_Vertical_screw_centered -> Potentiometer_THT:Potentiometer_Bourns_3296P_Horizontal
Connections:
- net GND: now also U1.5 (+); no longer U1.3 (+)
- net OCTAVE: now also U1.3 (+); no longer U1.5 (+)
- net at R25.1, R26.1, R28.2: now also U1.6 (-); no longer U1.2 (-)
- net at R28.1, R30.2: now also U1.7; no longer U1.1
- new net: R4.2, U1.1, U1.2 (-)
Other:
- moved on the sheet: U1A, U1B
Changed lines of the file:
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@@
     (property "Reference" "RV2" (id 0) (at 44.45 22.6822 90))
     (property "Value" "10k" (id 1) (at 44.45 24.9936 90))
-    (property "Footprint" "ao_tht:Potentiometer_Bourns_3296W_Vertical_screw_centered" (id 2) (at 44.45 27.94 0)
+    (property "Footprint" "Potentiometer_THT:Potentiometer_Bourns_3296P_Horizontal" (id 2) (at 44.45 27.94 0)
       (effects (font (size 1.27 1.27)) hide)
     )
@@
     (in_bom yes) (on_board yes)
     (property "Reference" "RV5" (id 0) (at 104.14 111.5822 90))
-    (property "Value" "20k" (id 1) (at 104.14 113.8936 90))
-    (property "Footprint" "ao_tht:Potentiometer_Bourns_3296W_Vertical_screw_centered" (id 2) (at 104.14 116.84 0)
+    (property "Value" "10k" (id 1) (at 104.14 113.8936 90))
+    (property "Footprint" "Potentiometer_THT:Potentiometer_Bourns_3296P_Horizontal" (id 2) (at 104.14 116.84 0)
       (effects (font (size 1.27 1.27)) hide)
     )
@@
     (in_bom yes) (on_board yes)
     (property "Reference" "RV6" (id 0) (at 104.14 125.5522 90))
-    (property "Value" "20k" (id 1) (at 104.14 127.8636 90))
-    (property "Footprint" "ao_tht:Potentiometer_Bourns_3296W_Vertical_screw_centered" (id 2) (at 104.14 130.81 0)
+    (property "Value" "10k" (id 1) (at 104.14 127.8636 90))
+    (property "Footprint" "Potentiometer_THT:Potentiometer_Bourns_3296P_Horizontal" (id 2) (at 104.14 130.81 0)
       (effects (font (size 1.27 1.27)) hide)
     )
@@
     (pin "2")
   )
-  (symbol (lib_id "ao_symbols:TL072") (at 217.17 121.92 0) (unit 1)
-    (in_bom yes) (on_board yes)
-    (property "Reference" "U1" (id 0) (at 217.17 112.5982 0))
-    (property "Value" "TL072" (id 1) (at 217.17 114.9096 0))
-    (property "Footprint" "ao_tht:DIP-8_W7.62mm_Socket_LongPads" (id 2) (at 215.9 119.38 0)
-      (effects (font (size 1.27 1.27)) hide)
-    )
-    (property "Datasheet" "" (id 3) (at 218.44 116.84 0)
-      (effects (font (size 1.27 1.27)) hide)
-    )
-    (property "Vendor" "Tayda" (id 4) (at 217.17 121.92 0)
-      (effects (font (size 1.27 1.27)) hide)
-    )
-    (property "SKU" "A-037" (id 5) (at 217.17 121.92 0)
+  (symbol (lib_id "ao_symbols:TL072") (at 45.72 120.65 0) (unit 1)
+    (in_bom yes) (on_board yes)
+    (property "Reference" "U1" (id 0) (at 45.72 111.3282 0))
+    (property "Value" "TL072" (id 1) (at 45.72 113.6396 0))
+    (property "Footprint" "ao_tht:DIP-8_W7.62mm_Socket_LongPads" (id 2) (at 44.45 118.11 0)
+      (effects (font (size 1.27 1.27)) hide)
+    )
+    (property "Datasheet" "" (id 3) (at 46.99 115.57 0)
+      (effects (font (size 1.27 1.27)) hide)
+    )
+    (property "Vendor" "Tayda" (id 4) (at 45.72 120.65 0)
+      (effects (font (size 1.27 1.27)) hide)
+    )
+    (property "SKU" "A-037" (id 5) (at 45.72 120.65 0)
       (effects (font (size 1.27 1.27)) hide)
     )
@@
       (effects (font (size 1.27 1.27)) (justify right))
     )
-    (property "Value" "50k" (id 1) (at 239.522 129.413 0)
+    (property "Value" "10k" (id 1) (at 239.522 129.413 0)
       (effects (font (size 1.27 1.27)) (justify right))
     )
-    (property "Footprint" "ao_tht:Potentiometer_Bourns_3296W_Vertical_screw_centered" (id 2) (at 241.3 128.27 0)
+    (property "Footprint" "Potentiometer_THT:Potentiometer_Bourns_3296P_Horizontal" (id 2) (at 241.3 128.27 0)
       (effects (font (size 1.27 1.27)) hide)
     )
@@
     (pin "1")
   )
-  (symbol (lib_id "ao_symbols:TL072") (at 45.72 120.65 0) (unit 2)
-    (in_bom yes) (on_board yes)
-    (property "Reference" "U1" (id 0) (at 45.72 111.3282 0))
-    (property "Value" "TL072" (id 1) (at 45.72 113.6396 0))
-    (property "Footprint" "ao_tht:DIP-8_W7.62mm_Socket_LongPads" (id 2) (at 44.45 118.11 0)
-      (effects (font (size 1.27 1.27)) hide)
-    )
-    (property "Datasheet" "" (id 3) (at 46.99 115.57 0)
-      (effects (font (size 1.27 1.27)) hide)
-    )
-    (property "Vendor" "Tayda" (id 4) (at 45.72 120.65 0)
-      (effects (font (size 1.27 1.27)) hide)
-    )
-    (property "SKU" "A-037" (id 5) (at 45.72 120.65 0)
-      (effects (font (size 1.27 1.27)) hide)
-    )
+  (symbol (lib_id "ao_symbols:TL072") (at 217.17 121.92 0) (unit 2)
+    (in_bom yes) (on_board yes)
+    (property "Reference" "U1" (id 0) (at 217.17 112.5982 0))
+    (property "Value" "TL072" (id 1) (at 217.17 114.9096 0))
+    (property "Footprint" "ao_tht:DIP-8_W7.62mm_Socket_LongPads" (id 2) (at 215.9 119.38 0)
+      (effects (font (size 1.27 1.27)) hide)
+    )
+    (property "Datasheet" "" (id 3) (at 218.44 116.84 0)
+      (effects (font (size 1.27 1.27)) hide)
+    )
+    (property "Vendor" "Tayda" (id 4) (at 217.17 121.92 0)
+      (effects (font (size 1.27 1.27)) hide)
+    )
+    (property "SKU" "A-037" (id 5) (at 217.17 121.92 0)
+      (effects (font (size 1.27 1.27)) hide)
+    )

Commit message: Correct slide switch footprint; use TO-92 wide for regulator
Parts:
- U6: footprint Package_TO_SOT_THT:TO-92_Inline -> ao_tht:TO-92_Inline_Wide
Changed lines of the file:
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@@
     (property "Reference" "U6" (id 0) (at 241.3 47.1932 0))
     (property "Value" "L79L05_TO92" (id 1) (at 241.3 49.5046 0))
-    (property "Footprint" "Package_TO_SOT_THT:TO-92_Inline" (id 2) (at 241.3 48.26 0)
+    (property "Footprint" "ao_tht:TO-92_Inline_Wide" (id 2) (at 241.3 48.26 0)
       (effects (font (size 1.27 1.27) italic) hide)
     )
