File: Hardware/PCB/sidekickvco/sidekickvco_main.kicad_sch (KiCad schematic)
At the start: 55 parts, among them U1 TL072, U3 AS3340A, U4 LM4040BIZ-5, U5 LM4040BIZ-5, U6 L79L05_TO92

Commit message: Pre prototype revisions, README revision
Parts:
- R1: renamed from R27; value 300k -> 30k
- R2: renamed from R31; value 300k -> 30k
- renumbered C11 to C10, C12 to C11, C13 to C12, C10 to C4, C20 to C5, R6 to R10, R7 to R11, R18 to R12, R10 to R13, R11 to R14, R13 to R15, R14 to R16, R15 to R17, R19 to R18, R20 to R19, R16 to R20, R17 to R21, R28 to R27, R29 to R28, R30 to R29, R1 to R3, R2 to R4, R3 to R5, R8 to R6, R9 to R7, R4 to R8, R5 to R9, RV2 to RV1, RV5 to RV2, RV6 to RV3, RV9 to RV4, TP2 to TP1, TP4 to TP2, TP6 to TP3, U3 to U2, U4 to U3, U5 to U4, U6 to U5
Other:
- note added: "Match these with octave switch 10k"
- note removed: "Does this work? Or do the CVs need to be summed outside the 3340?"
- note removed: "Make this 470k?"
- note removed: "Match these with octave switch 100k"

Commit message: Fix nuked footprints; update trimmer footprints
Parts:
- C1, C2, C3, C6: value 100nF -> (none); footprint ao_tht:C_Disc_D3.0mm_W1.6mm_P2.50mm -> (none)
- C10, C12, C4, C5, C8: value 10nF -> (none); footprint ao_tht:C_Rect_L7.2mm_W2.5mm_P5.00mm_FKS2_FKP2_MKS2_MKP2 -> (none)
- C11, C7: value 100nF -> (none); footprint ao_tht:C_Rect_L7.2mm_W2.5mm_P5.00mm_FKS2_FKP2_MKS2_MKP2 -> (none)
- C9: value 1nF -> (none); footprint Capacitor_THT:C_Rect_L7.2mm_W4.5mm_P5.00mm_FKS2_FKP2_MKS2_MKP2 -> (none)
- D1, D2: value 1N4148 -> (none); footprint ao_tht:D_DO-35_SOD27_P7.62mm_Horizontal -> (none)
- R1, R2: value 30k -> (none); footprint ao_tht:R_Axial_DIN0207_L6.3mm_D2.5mm_P10.16mm_Horizontal -> (none)
- R10, R25, R26, R27, R6, R7, R8, R9: value 100k -> (none); footprint ao_tht:R_Axial_DIN0207_L6.3mm_D2.5mm_P10.16mm_Horizontal -> (none)
- R11: value 470k -> (none); footprint ao_tht:R_Axial_DIN0207_L6.3mm_D2.5mm_P10.16mm_Horizontal -> (none)
- R12, R13, R18, R3: value 1M -> (none); footprint ao_tht:R_Axial_DIN0207_L6.3mm_D2.5mm_P10.16mm_Horizontal -> (none)
- R14, R17: value 470R -> (none); footprint ao_tht:R_Axial_DIN0207_L6.3mm_D2.5mm_P10.16mm_Horizontal -> (none)
- R15: value 1.8k -> (none); footprint ao_tht:R_Axial_DIN0207_L6.3mm_D2.5mm_P10.16mm_Horizontal -> (none)
- R16: value 1.5M -> (none); footprint ao_tht:R_Axial_DIN0207_L6.3mm_D2.5mm_P10.16mm_Horizontal -> (none)
- R19, R21, R28: value 47k -> (none); footprint ao_tht:R_Axial_DIN0207_L6.3mm_D2.5mm_P10.16mm_Horizontal -> (none)
- R20, R5: value 5.6k -> (none); footprint ao_tht:R_Axial_DIN0207_L6.3mm_D2.5mm_P10.16mm_Horizontal -> (none)
- R22: value 10k -> (none); footprint ao_tht:R_Axial_DIN0207_L6.3mm_D2.5mm_P10.16mm_Horizontal -> (none)
- R23, R24: value 1k -> (none); footprint ao_tht:R_Axial_DIN0207_L6.3mm_D2.5mm_P10.16mm_Horizontal -> (none)
- R29: value 20k -> (none); footprint ao_tht:R_Axial_DIN0207_L6.3mm_D2.5mm_P10.16mm_Horizontal -> (none)
- R4: value 24k -> (none); footprint ao_tht:R_Axial_DIN0207_L6.3mm_D2.5mm_P10.16mm_Horizontal -> (none)
- RV1, RV2, RV3, RV4: value 10k -> (none); footprint Potentiometer_THT:Potentiometer_Bourns_3296P_Horizontal -> (none)
- TP1: value +5VREF -> (none); footprint ao_tht:TestPoint_THTPad_D1.5mm_Drill0.7mm -> (none)
- TP2: value -5VREF -> (none); footprint ao_tht:TestPoint_THTPad_D1.5mm_Drill0.7mm -> (none)
- TP3: value -5V -> (none); footprint ao_tht:TestPoint_THTPad_D1.5mm_Drill0.7mm -> (none)
- U1: value TL072 -> (none); footprint ao_tht:DIP-8_W7.62mm_Socket_LongPads -> (none)
- U2: value AS3340A -> (none); footprint ao_tht:DIP-16_W7.62mm_Socket_LongPads -> (none)
- U3, U4: value LM4040BIZ-5 -> (none); footprint ao_tht:TO-92_Inline_Wide -> (none)
- U5: value L79L05_TO92 -> (none); footprint ao_tht:TO-92_Inline_Wide -> (none)

Commit message: Post prototype updates
Parts:
- C1, C2, C3, C6: value (none) -> 100nF; footprint (none) -> ao_tht:C_Disc_D3.0mm_W1.6mm_P2.50mm
- C10, C12, C4, C5, C8: value (none) -> 10nF; footprint (none) -> ao_tht:C_Rect_L7.2mm_W2.5mm_P5.00mm_FKS2_FKP2_MKS2_MKP2; SKU (none) -> A-559
- C11, C7: value (none) -> 100nF; footprint (none) -> ao_tht:C_Rect_L7.2mm_W2.5mm_P5.00mm_FKS2_FKP2_MKS2_MKP2; SKU (none) -> A-564
- C9: value (none) -> 1nF; footprint (none) -> Capacitor_THT:C_Rect_L7.2mm_W4.5mm_P5.00mm_FKS2_FKP2_MKS2_MKP2; SKU (none) -> FKP2G011001D00HSSD; Vendor Tayda -> Digi-Key
- D1, D2: value (none) -> 1N4148; footprint (none) -> ao_tht:D_DO-35_SOD27_P7.62mm_Horizontal
- R1, R2: value (none) -> 30k; footprint (none) -> ao_tht:R_Axial_DIN0207_L6.3mm_D2.5mm_P10.16mm_Horizontal
- R10, R25, R26, R27, R6, R7, R8, R9: value (none) -> 100k; footprint (none) -> ao_tht:R_Axial_DIN0207_L6.3mm_D2.5mm_P10.16mm_Horizontal
- R11: value (none) -> 470k; footprint (none) -> ao_tht:R_Axial_DIN0207_L6.3mm_D2.5mm_P10.16mm_Horizontal
- R12, R13, R18, R3: value (none) -> 1M; footprint (none) -> ao_tht:R_Axial_DIN0207_L6.3mm_D2.5mm_P10.16mm_Horizontal
- R14, R17: value (none) -> 470R; footprint (none) -> ao_tht:R_Axial_DIN0207_L6.3mm_D2.5mm_P10.16mm_Horizontal
- R15: value (none) -> 1.8k; footprint (none) -> ao_tht:R_Axial_DIN0207_L6.3mm_D2.5mm_P10.16mm_Horizontal
- R16: value (none) -> 1.5M; footprint (none) -> ao_tht:R_Axial_DIN0207_L6.3mm_D2.5mm_P10.16mm_Horizontal
- R19, R21, R28: value (none) -> 47k; footprint (none) -> ao_tht:R_Axial_DIN0207_L6.3mm_D2.5mm_P10.16mm_Horizontal
- R20, R5: value (none) -> 5.6k; footprint (none) -> ao_tht:R_Axial_DIN0207_L6.3mm_D2.5mm_P10.16mm_Horizontal
- R22: value (none) -> 10k; footprint (none) -> ao_tht:R_Axial_DIN0207_L6.3mm_D2.5mm_P10.16mm_Horizontal
- R23, R24: value (none) -> 1k; footprint (none) -> ao_tht:R_Axial_DIN0207_L6.3mm_D2.5mm_P10.16mm_Horizontal
- R29: value (none) -> 20k; footprint (none) -> ao_tht:R_Axial_DIN0207_L6.3mm_D2.5mm_P10.16mm_Horizontal
- R4: value (none) -> 24k; footprint (none) -> ao_tht:R_Axial_DIN0207_L6.3mm_D2.5mm_P10.16mm_Horizontal
- RV1, RV2, RV3: value (none) -> 10k; footprint (none) -> ao_tht:Potentiometer_Bourns_3296P_Horizontal; SKU (none) -> CT94EP103-ND; Vendor Tayda -> Digi-Key
- RV4: value (none) -> 50k; footprint (none) -> ao_tht:Potentiometer_Bourns_3296P_Horizontal; SKU (none) -> CT94EP503-ND; Vendor Tayda -> Digi-Key
- TP1: value (none) -> +5VREF; footprint (none) -> ao_tht:TestPoint_THTPad_D1.5mm_Drill0.7mm
- TP2: value (none) -> -5VREF; footprint (none) -> ao_tht:TestPoint_THTPad_D1.5mm_Drill0.7mm
- TP3: value (none) -> -5V; footprint (none) -> ao_tht:TestPoint_THTPad_D1.5mm_Drill0.7mm
- U1: value (none) -> TL072; footprint (none) -> ao_tht:DIP-8_W7.62mm_Socket_LongPads
- U2: value (none) -> AS3340A; footprint (none) -> ao_tht:DIP-16_W7.62mm_Socket_LongPads; Vendor (none) -> CabinTech Global
- U3, U4: value (none) -> LM4040BIZ-5; footprint (none) -> ao_tht:TO-92_Inline_Wide; SKU (none) -> LM4040BIZ-5/NOPB-ND; Vendor (none) -> Digi-Key
- U5: value (none) -> L79L05_TO92; footprint (none) -> ao_tht:TO-92_Inline_Wide; SKU (none) -> A-4676; Vendor (none) -> Tayda

Commit message: Fix lin FM input, add howitworks
Parts:
- removed R7: 100k, ao_tht:R_Axial_DIN0207_L6.3mm_D2.5mm_P10.16mm_Horizontal, symbol ao_symbols:R
Connections:
- net GND: now also R6.2
- net LINK_IN_FM: now also C5.2
- net LIN_FM_IN: now also C4.2, R6.1; no longer R6.2
Other:
- moved on the sheet: C4, C5, R12, R13

Commit message: Restore resistor
Parts:
- added R7: 100k, ao_tht:R_Axial_DIN0207_L6.3mm_D2.5mm_P10.16mm_Horizontal, symbol ao_symbols:R
Connections:
- net GND: now also R7.2
- net LINK_IN_FM: now also R7.1
Changed lines of the file:
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@@
   (junction (at 241.3 121.92) (diameter 0) (color 0 0 0 0)
+  )
+  (junction (at 68.58 99.06) (diameter 0) (color 0 0 0 0)
   )
   (junction (at 40.64 52.07) (diameter 0) (color 0 0 0 0)
@@
     (stroke (width 0) (type default) (color 0 0 0 0))
   )
+  (wire (pts (xy 68.58 99.06) (xy 68.58 100.33))
+    (stroke (width 0) (type default) (color 0 0 0 0))
+  )
   (wire (pts (xy 105.41 49.53) (xy 104.14 49.53))
     (stroke (width 0) (type default) (color 0 0 0 0))
@@
     (stroke (width 0) (type default) (color 0 0 0 0))
   )
-  (wire (pts (xy 62.23 99.06) (xy 78.74 99.06))
+  (wire (pts (xy 62.23 99.06) (xy 68.58 99.06))
     (stroke (width 0) (type default) (color 0 0 0 0))
   )
@@
   )
   (wire (pts (xy 251.46 53.34) (xy 248.92 53.34))
+    (stroke (width 0) (type default) (color 0 0 0 0))
+  )
+  (wire (pts (xy 68.58 99.06) (xy 78.74 99.06))
     (stroke (width 0) (type default) (color 0 0 0 0))
   )
@@
     (pin "1")
   )
+  (symbol (lib_id "power:GND") (at 68.58 107.95 0) (unit 1)
+    (in_bom yes) (on_board yes) (fields_autoplaced)
+    (property "Reference" "#PWR?" (id 0) (at 68.58 114.3 0)
+      (effects (font (size 1.27 1.27)) hide)
+    )
+    (property "Value" "GND" (id 1) (at 68.58 112.3934 0))
+    (property "Footprint" "" (id 2) (at 68.58 107.95 0)
+      (effects (font (size 1.27 1.27)) hide)
+    )
+    (property "Datasheet" "" (id 3) (at 68.58 107.95 0)
+      (effects (font (size 1.27 1.27)) hide)
+    )
+    (pin "1")
+  )
   (symbol (lib_id "ao_symbols:TL072") (at 217.17 121.92 0) (unit 2)
     (in_bom yes) (on_board yes)
@@
       (effects (font (size 1.27 1.27)) hide)
     )
+    (pin "1")
+    (pin "2")
+  )
+  (symbol (lib_id "ao_symbols:R") (at 68.58 104.14 0) (unit 1)
+    (in_bom yes) (on_board yes) (fields_autoplaced)
+    (property "Reference" "R7" (id 0) (at 70.358 103.3053 0)
+      (effects (font (size 1.27 1.27)) (justify left))
+    )
+    (property "Value" "100k" (id 1) (at 70.358 105.8422 0)
+      (effects (font (size 1.27 1.27)) (justify left))
+    )
+    (property "Footprint" "ao_tht:R_Axial_DIN0207_L6.3mm_D2.5mm_P10.16mm_Horizontal" (id 2) (at 66.802 104.14 90)
+      (effects (font (size 1.27 1.27)) hide)
+    )
+    (property "Datasheet" "" (id 3) (at 68.58 104.14 0)
+      (effects (font (size 1.27 1.27)) hide)
+    )
+    (property "Vendor" "Tayda" (id 4) (at 68.58 104.14 0)
+      (effects (font (size 1.27 1.27)) hide)
+    )
