File: Hardware/PCB/sidekickvco/sidekickvco.kicad_pcb (KiCad board)
At the start: 2 copper layers, 269 x 172 mm, 163 parts, among them J1 Conn_01x09, J10 Conn_01x03, J11 Conn_01x03, J12 3_pin_Molex_connector, J13 Wire pads, J14 Conn_01x01, J15 Conn_01x01, J16 Conn_01x01, J17 Conn_02x04_Odd_Even, J18 AudioJack2, J19 AudioJack2, J2 Conn_01x03, J20 AudioJack2, J21 AudioJack2, J22 AudioJack2, J23 Synth_power_2x5, J24 AudioJack2, J25 AudioJack2, J26 AudioJack2, J27 AudioJack2, J28 AudioJack2, J3 Conn_01x03, J4 3_pin_Molex_header, J5 Wire pads, J6 Conn_01x01, J7 Conn_01x01, J8 Conn_01x01, J9 Conn_01x09, Q1 2N3904, Q2 2N3904, SW1 SW_Rotary12, SW2 SW_DP3T, U1 TL074, U2 TL072, U3 AS3340A, U4 LM4040BIZ-5, U5 LM4040BIZ-5, U6 L79L05_TO92, U7 TL074

Commit message: Initial version of circuit and layout
Parts:
- removed B1, B2: Board, ao_tht:Board_Marker
- removed C4, C5: 100nF, ao_tht:C_Disc_D3.0mm_W1.6mm_P2.50mm
- removed H1, H2, H3, H4, H5, H6: MountingHole, ao_tht:MountingHole_3.2mm_M3
- removed J10, J11: Conn_01x03, Connector_PinSocket_2.54mm:PinSocket_1x03_P2.54mm_Vertical
- removed J12: 3_pin_Molex_connector, ao_tht:Molex_KK-254_AE-6410-03A_1x03_P2.54mm_Vertical
- removed J13: Wire pads, Connector_Wire:SolderWire-0.5sqmm_1x01_D0.9mm_OD2.1mm
- removed J14, J15, J7, J8: Conn_01x01, herovco:SolderWire-round_1x01_D0.9mm_OD2.1mm
- removed J25, J27, J28: AudioJack2, ao_tht:Jack_6.35mm_PJ_629HAN
- removed J9: Conn_01x09, Connector_PinSocket_2.54mm:PinSocket_1x09_P2.54mm_Vertical
- removed R12: 10k, ao_tht:R_Axial_DIN0207_L6.3mm_D2.5mm_P10.16mm_Horizontal
- removed R21: 100k, ao_tht:R_Axial_DIN0207_L6.3mm_D2.5mm_P10.16mm_Horizontal
- removed R32, R33, R34, R35, R36, R37, R38, R39, R40, R41: 10k 1/8W, ao_tht:R_Axial_DIN0207_L6.3mm_D2.5mm_P10.16mm_Horizontal
- removed RV1, RV3, RV4, RV7, RV8: 100k, ao_tht:Potentiometer_Alpha_RD901F-40-00D_Single_Vertical_centered
- removed SW1: SW_Rotary12, ao_tht:Rotary_Switch
- removed TP1: +12V, ao_tht:TestPoint_THTPad_D1.5mm_Drill0.7mm
- removed TP3: -12V, ao_tht:TestPoint_THTPad_D1.5mm_Drill0.7mm
- removed TP5: GND, ao_tht:TestPoint_THTPad_D1.5mm_Drill0.7mm
- removed the U1 at (105.4, 115.6)
- added C20: 10nF, ao_tht:C_Rect_L7.2mm_W2.5mm_P5.00mm_FKS2_FKP2_MKS2_MKP2, F.Cu at (101.7, 37.9)
- C1, C10, C11, C12, C13, C14, C15, C16, C17, C18, C19, C2, C3, C6, C7, C8, C9, D1, D2, D3, D4, GRAF3, GRAF4, J17, J23, J4, Q1, Q2, R1, R11, R13, R14, R15, R16, R17, R18, R19, R2, R20, R22, R23, R24, R26, R28, R29, R3, R30, R4, R42, R43, R44, R45, R46, R47, R48, R49, R5, R50, R51, R52, R53, R54, R55, R56, R57, R58, R59, R6, R60, R61, R62, R63, R64, R65, R66, R67, R7, R8, RV10, RV11, RV12, U3, U4, U5, U6, U7: moved to F.Cu
- J1: value Conn_01x09 -> 3_pin_Molex_header; footprint Connector_PinHeader_2.54mm:PinHeader_1x09_P2.54mm_Vertical -> ao_tht:Molex_KK-254_AE-6410-03A_1x03_P2.54mm_Vertical; moved to F.Cu
- J16: value Conn_01x01 -> Wire pad; footprint herovco:SolderWire-round_1x01_D0.9mm_OD2.1mm -> Connector_Wire:SolderWire-0.5sqmm_1x01_D0.9mm_OD2.1mm
- J18, J22, J24, J26: footprint ao_tht:Jack_6.35mm_PJ_629HAN -> ao_tht:Jack_6.35mm_TE-CK-6.35-29B_Horizontal
- J19, J20, J21: value AudioJack2 -> Wire pad; footprint ao_tht:Jack_6.35mm_PJ_629HAN -> Connector_Wire:SolderWire-0.5sqmm_1x01_D0.9mm_OD2.1mm
- J2: value Conn_01x03 -> 4_pin_Molex_header; footprint Connector_PinHeader_2.54mm:PinHeader_1x03_P2.54mm_Vertical -> Connector_Molex:Molex_KK-254_AE-6410-04A_1x04_P2.54mm_Vertical; moved to F.Cu
- J3: value Conn_01x03 -> 2_pin_Molex_header; footprint Connector_PinHeader_2.54mm:PinHeader_1x03_P2.54mm_Vertical -> ao_tht:Molex_KK-254_AE-6410-02A_1x02_P2.54mm_Vertical; moved to F.Cu
- J5: value Wire pads -> 2_pin_Molex_header; footprint Connector_Wire:SolderWire-0.5sqmm_1x01_D0.9mm_OD2.1mm -> ao_tht:Molex_KK-254_AE-6410-02A_1x02_P2.54mm_Vertical
- J6: value Conn_01x01 -> 2_pin_Molex_header; footprint herovco:SolderWire-round_1x01_D0.9mm_OD2.1mm -> ao_tht:Molex_KK-254_AE-6410-02A_1x02_P2.54mm_Vertical
- R10: value 100k -> 1M; moved to F.Cu
- R25: value 240k -> 100k; moved to F.Cu
- R27, R31: value 10k -> 300k; moved to F.Cu
- R9: value 10k -> 100k; moved to F.Cu
- TP2, TP4, TP6, TP7, TP8, TP9: moved to B.Cu
- U1: renamed from U2; moved to F.Cu
- moved J19 247.9 mm to (24.2, 111.5), turned to 0 degrees
- moved J21 234.7 mm to (12.8, 111.5), turned to 0 degrees
- moved TP7 201.5 mm to (78.8, 170.0)
- moved TP8 201.5 mm to (78.8, 185.2)
- moved TP9 201.5 mm to (78.8, 177.6)
- moved RV10 193.4 mm to (84.0, 121.7)
- moved RV11 193.4 mm to (84.0, 134.4)
- moved RV12 193.4 mm to (84.0, 156.0)
- moved R62 175.2 mm to (96.5, 114.1), turned to 0 degrees
- moved Q1 175.0 mm to (96.6, 139.5), turned to 0 degrees
- moved Q2 175.0 mm to (96.6, 126.8), turned to 0 degrees
- moved R42 175.0 mm to (96.6, 121.7), turned to 0 degrees
- moved R43 175.0 mm to (96.6, 143.3), turned to 0 degrees
- moved R48 175.0 mm to (96.6, 117.9), turned to 0 degrees
- moved R49 175.0 mm to (96.6, 154.7), turned to 0 degrees
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Connections:
- net /Front PCB/CENTER_FREQ renamed /Main PCB/CENTER_FREQ
- net /Front PCB/HI_FREQ_TRACK renamed /Main PCB/HI_FREQ_TRACK
- net /Jacks, power, etc/SIN renamed SIN
- C10 pad 2: /Front PCB/LINK_OUT_FM -> Net-(C10-Pad2)
- C12 pad 2: /Front PCB/SOFT_SYNC_OFF -> /Main PCB/SOFT_SYNC_OFF
- C14 pad 1: +12V_1 -> +12V
- C14 pad 2: GND1 -> GND
- C15 pad 1: GND1 -> GND
- C15 pad 2: -12V_1 -> -12V
- C16 pad 1: +12V_1 -> +12V
- C16 pad 2: GND1 -> GND
- C17 pad 1: GND1 -> GND
- C17 pad 2: -12V_1 -> -12V
- C18 pad 1: /Outputs and sin/LINK_OUT_SAW -> Net-(C18-Pad1)
- C7 pad 1: /Front PCB/SYNCA -> /Main PCB/SYNCA
- C7 pad 2: /Front PCB/SYNC -> /Main PCB/LINK_IN_SYNC
- D3 pad 1: +12V_1 -> +12V
- D4 pad 2: -12V_1 -> -12V
- J1 pad 1: GND -> -5V_REF
- J1 pad 2: -12V -> /Main PCB/FINE_TUNE
- J1 pad 3: +12V -> +5V_REF
- J16 pad 1: /Octave and sync switches/HARD_SYNCA_P -> /Panel mounted components/SYNCA_P
- J17 pad 1: /Outputs and sin/LINK_OUT_SAW -> /Main PCB/LINK_IN_SYNC
- J17 pad 2: GND1 -> GND
- J17 pad 3: /LINK_OUT_FM_B -> /Main PCB/LINK_IN_FM
- J17 pad 4: GND1 -> GND
- J17 pad 5: /LINK_OUT_PW_B -> /Main PCB/LINK_IN_PW
- J17 pad 6: GND1 -> GND
- J17 pad 7: /LINK_OUT_CV_B -> /Main PCB/LINK_IN_CV
- J17 pad 8: GND1 -> GND
- J18 pad S: GND1 -> GND
- J18 pad T: /Jacks, power, etc/PWMIN_J -> PWMIN
- J2 pad 1: /Front PCB/TRIANGLE_OUT -> /Main PCB/SYNCA
- J2 pad 2: /Front PCB/PULSE_OUT -> /Main PCB/SOFT_SYNCA
- J2 pad 3: /Front PCB/SAW_OUT -> /Main PCB/SOFT_SYNC_OFF
- J22 pad S: GND1 -> GND
- J22 pad T: /Jacks, power, etc/V_OCT_J -> V_OCT
- J23 pad 3: GND1 -> GND
- J23 pad 4: GND1 -> GND
- J23 pad 5: GND1 -> GND
- J23 pad 6: GND1 -> GND
- J23 pad 7: GND1 -> GND
- J23 pad 8: GND1 -> GND
- J24 pad S: GND1 -> GND
- J26 pad S: GND1 -> GND
- J3 pad 1: /Front PCB/LINK_OUT_FM -> GND
- J3 pad 2: /Front PCB/LINK_OUT_PW -> /Main PCB/LIN_FM_IN
- J4 pad 1: /Front PCB/+5V_REF -> /Main PCB/+2V_REF
- J4 pad 2: /Front PCB/OCTAVE -> /Main PCB/OCTAVE
- J4 pad 3: /Front PCB/-5V_REF -> /Main PCB/-2V_REF
- J5 pad 1: /Front PCB/SYNCA -> GND
- J6 pad 1: /Front PCB/SOFT_SYNCA -> GND
- R1 pad 1: /Front PCB/PULSE_OUT -> PULSE_OUT
- R10 pad 1: Net-(R10-Pad1) -> LIN_FM
- R10 pad 2: Net-(R10-Pad2) -> Net-(C20-Pad1)
- R16 pad 2: /Front PCB/HARD_SYNCA -> /Main PCB/HARD_SYNCA
- R17 pad 2: /Front PCB/SOFT_SYNCA -> /Main PCB/SOFT_SYNCA
- R23 pad 2: /Front PCB/+5V_REF -> +5V_REF
- R24 pad 1: /Front PCB/-5V_REF -> -5V_REF
- R25 pad 2: /Front PCB/PULSE_WIDTH -> /Main PCB/LINK_IN_PW
- R26 pad 2: /Front PCB/PWM -> PWMIN
- R27 pad 1: Net-(R27-Pad1) -> +5V_REF
- R27 pad 2: Net-(R27-Pad2) -> /Main PCB/+2V_REF
- R28 pad 1: Net-(R27-Pad2) -> Net-(R28-Pad1)
- R30 pad 2: Net-(R27-Pad2) -> Net-(R28-Pad1)
- R31 pad 1: /Front PCB/LINK_OUT_PW -> -5V_REF
- R31 pad 2: Net-(R27-Pad1) -> /Main PCB/-2V_REF
- R4 pad 1: Net-(R10-Pad2) -> CV_NODE
- R43 pad 2: GND1 -> GND
- R44 pad 1: +12V_1 -> +12V
- R46 pad 1: +12V_1 -> +12V
- R47 pad 1: -12V_1 -> -12V
- R48 pad 2: GND1 -> GND
- R49 pad 2: GND1 -> GND
- R5 pad 1: Net-(R10-Pad2) -> CV_NODE
- R5 pad 2: /Front PCB/V_OCT -> V_OCT
- R52 pad 2: /Outputs and sin/SAW_OUT_S -> SAW_OUT
- R53 pad 2: /Outputs and sin/PULSE_OUT_S -> PULSE_OUT
- R54 pad 2: GND1 -> GND
- R55 pad 2: GND1 -> GND
- R56 pad 2: +12V_1 -> +12V
- R57 pad 2: +12V_1 -> +12V
- R58 pad 2: +12V_1 -> +12V
- R59 pad 2: GND1 -> GND
- R6 pad 1: Net-(R10-Pad2) -> CV_NODE
- R6 pad 2: /Front PCB/V_OCT2 -> /Main PCB/LINK_IN_CV
- R60 pad 2: GND1 -> GND
- R61 pad 2: GND1 -> GND
- R63 pad 1: /Outputs and sin/LINK_OUT_SAW -> Net-(C18-Pad1)
- R65 pad 1: TRI -> /Outputs and sin/TRI
- R66 pad 1: SAW -> /Outputs and sin/SAW
- R66 pad 2: /Outputs and sin/LINK_OUT_SAW -> Net-(C18-Pad1)
- R7 pad 1: Net-(R10-Pad2) -> CV_NODE
- R7 pad 2: /Front PCB/FINE_TUNE -> /Main PCB/FINE_TUNE
- R8 pad 1: Net-(R10-Pad2) -> Net-(C10-Pad2)
- R8 pad 2: /Front PCB/FREQ_CV -> /Main PCB/LIN_FM_IN
- R9 pad 2: Net-(R10-Pad1) -> /Main PCB/LINK_IN_FM
- RV12 pad 1: GND1 -> GND
- RV6 pad 3: /Front PCB/+5V_REF -> +5V_REF
- SW2 pad 1: /Octave and sync switches/HARD_SYNCA_P -> /Panel mounted components/HARD_SYNCA_P
- SW2 pad 2: /Octave and sync switches/SYNCA_P -> /Panel mounted components/SYNCA_P
- SW2 pad 4: /Octave and sync switches/SOFT_SYNCA_P -> /Panel mounted components/SOFT_SYNCA_P
- SW2 pad 5: /Octave and sync switches/SOFT_SYNC_OFF_P -> /Panel mounted components/SOFT_SYNC_OFF_P
- SW2 pad 6: /Octave and sync switches/SOFT_SYNCA_P -> /Panel mounted components/SOFT_SYNCA_P
- SW2 pad 7: /Octave and sync switches/SOFT_SYNC_OFF_P -> /Panel mounted components/SOFT_SYNC_OFF_P
- TP2 pad 1: /Front PCB/+5V_REF -> +5V_REF
- TP4 pad 1: /Front PCB/-5V_REF -> -5V_REF
- TP7 pad 1: +12V_1 -> +12V
- TP8 pad 1: -12V_1 -> -12V
- TP9 pad 1: GND1 -> GND
- U1 pad 1: Net-(R27-Pad2) -> Net-(R28-Pad1)
- U1 pad 5: GND -> /Main PCB/OCTAVE
- U1 pad 6: Net-(R27-Pad1) -> Net-(R4-Pad2)
- U1 pad 7: /Front PCB/LINK_OUT_PW -> Net-(R4-Pad2)
- U3 pad 10: /Front PCB/TRIANGLE_OUT -> TRIANGLE_OUT
- U3 pad 4: /Front PCB/PULSE_OUT -> PULSE_OUT
- U3 pad 8: /Front PCB/SAW_OUT -> SAW_OUT
- U4 pad 2: /Front PCB/+5V_REF -> +5V_REF
- U5 pad 3: /Front PCB/-5V_REF -> -5V_REF
- U7 pad 1: /Outputs and sin/LINK_OUT_SAW -> Net-(C18-Pad1)
- U7 pad 10: /Outputs and sin/TRIANGLE_OUT_S -> TRIANGLE_OUT
- U7 pad 11: -12V_1 -> -12V
- U7 pad 4: +12V_1 -> +12V
Routing:
- net TRI: track 170.7 -> 0.00 mm
- net /Front PCB/+5V_REF: track 161.2 -> 0.00 mm
- net +12V_1: track 158.7 -> 0.00 mm
- net PULSE_OUT: track 0.00 -> 128.9 mm
- net +5V_REF: track 0.00 -> 125.0 mm
- net /Front PCB/-5V_REF: track 109.8 -> 0.00 mm
- net SAW_OUT: track 0.00 -> 108.4 mm, vias 0 -> 1
- net PWMIN: track 0.00 -> 91.8 mm
- net -12V_1: track 87.2 -> 0.00 mm
- net TRIANGLE_OUT: track 0.00 -> 85.7 mm
- net -5V_REF: track 0.00 -> 75.1 mm
- net +12V: track 209.7 -> 280.7 mm
- net /Main PCB/LINK_IN_CV: track 0.00 -> 69.9 mm
- net Net-(R10-Pad2): track 69.3 -> 0.00 mm
- net -5V: track 81.9 -> 149.0 mm
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- removed copper zone on B.Cu, net GND1
- removed copper zone on F.Cu, net GND1
Other:
- board size 269 x 172 mm -> 169.5 x 170 mm
- board text removed: "+12 V"
- board text removed: "-12 V"
- board text removed: "Exp FM"
- board text removed: "FM"
- board text removed: "Fine tune"
- board text removed: "GND"
- board text removed: "Hero VCO front board"
- board text removed: "Lin FM"
- board text removed: "PW"
- board text removed: "Panel mounted"
- board text removed: "Pitch"
- board text removed: "Sin"
- board text removed: "Sync"
- board text removed: "Sync switch daughterboard"
- board text removed: "Tri"
- board text removed: "V/oct 1"
- board text removed: "V/oct 2"

Commit message: Daughterboard mounting
Parts:
- added GRAF1: board, sidekickvco:sidekick_daughterboard, F.Cu at (19.3, 118.0)
- added H1: MountingHole, ao_tht:MountingHole_3.2mm_M3, F.Cu at (28.8, 127.0)
- added H2: MountingHole, ao_tht:MountingHole_3.2mm_M3, F.Cu at (9.80, 109.0)
- J19, J20, J21: footprint Connector_Wire:SolderWire-0.5sqmm_1x01_D0.9mm_OD2.1mm -> sidekickvco:SolderWire-round_1x01_D0.9mm_OD2.1mm
- moved GRAF4 206.2 mm to (88.5, 166.1), turned to 90 degrees
- moved GRAF3 190.5 mm to (128.3, 189.0), turned to 90 degrees
- moved J21 16.7 mm to (29.3, 109.0)
- moved C12 14.9 mm to (150.0, 65.8)
- moved J20 5.68 mm to (25.5, 109.0)
- moved B3 5.15 mm to (18.4, 105.9)
- moved J19 3.59 mm to (21.7, 109.0)
- moved J16 2.84 mm to (17.9, 109.0)
Connections:
- J16 pad 1: /Panel mounted components/SYNCA_P -> /Panel mounted components/HARD_SYNCA_P
- J19 pad 1: /Panel mounted components/SOFT_SYNCA_P -> /Panel mounted components/SYNCA_P
- J2 pad 1: /Main PCB/SYNCA -> /Main PCB/HARD_SYNCA
- J2 pad 2: /Main PCB/SOFT_SYNCA -> /Main PCB/SYNCA
- J2 pad 4: /Main PCB/HARD_SYNCA -> /Main PCB/SOFT_SYNCA
- J21 pad 1: /Panel mounted components/HARD_SYNCA_P -> /Panel mounted components/SOFT_SYNCA_P
Routing:
- net /Main PCB/HARD_SYNCA: track 15.1 -> 7.82 mm
- net /Main PCB/SOFT_SYNC_OFF: track 7.37 -> 12.2 mm
- net /Panel mounted components/SOFT_SYNCA_P: track 14.0 -> 18.7 mm
- net /Panel mounted components/HARD_SYNCA_P: track 7.41 -> 12.1 mm
- net /Panel mounted components/SOFT_SYNC_OFF_P: track 18.8 -> 23.0 mm
- net /Panel mounted components/SYNCA_P: track 7.52 -> 11.6 mm
- net /Main PCB/SYNCA: track 34.3 -> 36.7 mm
- net /Main PCB/SOFT_SYNCA: track 9.72 -> 7.62 mm
Other:
- outline, holes or cut-outs redrawn
- board text added: "No power here Count the pins Power's I dunno maybe down by the bottom somewhere"
- board text added: "Rich Holmes CC0 1.0 Jan 2022 https://github.com/holmesrichards/sidekick"
- board text added: "Sidekick VCO"
- board text removed: "Back board"
- board text removed: "Hero VCO"
- board text removed: "No power here Count the pins Power's over there (gestures vaguely to the left)"
- board text removed: "Rich Holmes CC0 1.0 Jan 2022 https://github.com/holmesrichards/hero"

Commit message: Revise layout, add notes, BUILD.md
Parts:
- removed the GRAF1 at (103.8, 115.0)
- added B1: Board, ao_tht:Board_Marker, F.Cu at (125.8, 36.0)
- GRAF2: footprint herovco_panel:herovco_panel_holes -> sidekickvco:sidekick_panel_holes
- RV2: footprint ao_tht:Potentiometer_Bourns_3296W_Vertical_screw_centered -> Potentiometer_THT:Potentiometer_Bourns_3296P_Horizontal
- RV5, RV6: value 20k -> 10k; footprint ao_tht:Potentiometer_Bourns_3296W_Vertical_screw_centered -> Potentiometer_THT:Potentiometer_Bourns_3296P_Horizontal
- RV9: value 50k -> 10k; footprint ao_tht:Potentiometer_Bourns_3296W_Vertical_screw_centered -> Potentiometer_THT:Potentiometer_Bourns_3296P_Horizontal
- moved R29 68.1 mm to (163.9, 76.0), turned to 180 degrees
- moved J1 67.1 mm to (90.3, 49.3), turned to -90 degrees
- moved GRAF2 63.6 mm to (165.3, 112.0)
- moved C7 63.1 mm to (116.9, 107.7)
- moved GRAF4 62.5 mm to (145.3, 139.8)
- moved TP2 61.8 mm to (89.0, 40.4)
- moved R31 60.7 mm to (89.0, 63.3), turned to 0 degrees
- moved R27 60.6 mm to (89.0, 67.1), turned to 0 degrees
- moved U4 59.7 mm to (96.6, 40.8)
- moved U5 59.7 mm to (105.5, 40.8)
- moved J17 53.8 mm to (101.7, 103.9)
- moved R24 49.5 mm to (96.6, 45.5)
- moved TP4 49.3 mm to (89.0, 45.5)
- moved R4 49.0 mm to (97.9, 54.4), turned to 0 degrees
- moved R30 45.1 mm to (136.0, 46.8)
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- renumbered B3 to B2
Connections:
- U1 pad 1: Net-(R28-Pad1) -> Net-(R4-Pad2)
- U1 pad 2: Net-(R25-Pad1) -> Net-(R4-Pad2)
- U1 pad 3: GND -> /Main PCB/OCTAVE
- U1 pad 5: /Main PCB/OCTAVE -> GND
- U1 pad 6: Net-(R4-Pad2) -> Net-(R25-Pad1)
- U1 pad 7: Net-(R4-Pad2) -> Net-(R28-Pad1)
Routing:
- net +5V_REF: track 125.0 -> 204.4 mm
- net Net-(R28-Pad1): track 58.8 -> 9.95 mm
- net /Main PCB/LINK_IN_PW: track 16.4 -> 63.7 mm, vias 0 -> 1
- net -5V: track 149.0 -> 104.2 mm
- net Net-(C20-Pad1): track 50.9 -> 11.0 mm
- net /Main PCB/FINE_TUNE: track 45.7 -> 8.15 mm
- net +12V: track 280.7 -> 244.7 mm
- net SAW_OUT: track 108.3 -> 74.5 mm
- net Net-(R29-Pad1): track 86.3 -> 54.0 mm
- net -5V_REF: track 75.1 -> 43.5 mm
- net PULSE_OUT: track 128.9 -> 98.5 mm, vias 0 -> 1
- net /Main PCB/LINK_IN_CV: track 69.9 -> 39.7 mm
- net TRIANGLE_OUT: track 85.7 -> 56.5 mm
- net PWM_IN: track 99.4 -> 71.8 mm
- net HFT: track 87.9 -> 60.8 mm
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Other:
- board size 169.5 x 170 mm -> 169.5 x 163 mm
- board text added: "+2V"
- board text added: "-2V"
- board text added: "Sin"
- board text removed: "+5V"
- board text removed: "-5V"
- board text removed: "Lin FM CV"
- board text removed: "No power here Count the pins Power's I dunno maybe down by the bottom somewhere"
- board text removed: "Octave switch"
- board text removed: "Pulse width"
- board text removed: "RED STRIPE"

Commit message: Correct slide switch footprint; use TO-92 wide for regulator
Parts:
- U6: footprint Package_TO_SOT_THT:TO-92_Inline -> ao_tht:TO-92_Inline_Wide
- moved SW2 2.50 mm to (12.3, 121.3)
- moved U6 1.91 mm to (103.0, 84.2)
Connections:
- SW2 pad 1: /Panel mounted components/HARD_SYNCA_P -> /Panel mounted components/SOFT_SYNC_OFF_P
- SW2 pad 2: /Panel mounted components/SYNCA_P -> /Panel mounted components/SOFT_SYNCA_P
- SW2 pad 3: unconnected-(SW2-Pad3) -> /Panel mounted components/SOFT_SYNC_OFF_P
- SW2 pad 4: /Panel mounted components/SOFT_SYNCA_P -> unconnected-(SW2-Pad4)
- SW2 pad 5: /Panel mounted components/SOFT_SYNC_OFF_P -> /Panel mounted components/HARD_SYNCA_P
- SW2 pad 6: /Panel mounted components/SOFT_SYNCA_P -> /Panel mounted components/SYNCA_P
- SW2 pad 7: /Panel mounted components/SOFT_SYNC_OFF_P -> unconnected-(SW2-Pad7)
- SW2 pad 8: unconnected-(SW2-Pad8) -> /Panel mounted components/SOFT_SYNCA_P
Routing:
- net -5V: track 104.2 -> 104.7 mm

Commit message: 5 mm pitch for 330 pF
Parts:
- C18, C19: footprint ao_tht:C_Disc_D3.0mm_W1.6mm_P2.50mm -> ao_tht:C_Disc_D5.0mm_W2.5mm_P5.00mm
- moved C18 2.59 mm to (132.2, 166.2)
Routing:
- net Net-(C18-Pad1): track 35.7 -> 35.0 mm
