File: Hardware/PCB/sidekickvco/sidekickvco.kicad_pcb (KiCad board)
At the start: 2 copper layers, 169.5 x 163 mm, 123 parts, among them J1 3_pin_Molex_header, J16 Wire pad, J17 Conn_02x04_Odd_Even, J18 AudioJack2, J19 Wire pad, J2 4_pin_Molex_header, J20 Wire pad, J21 Wire pad, J22 AudioJack2, J23 Synth_power_2x5, J24 AudioJack2, J26 AudioJack2, J3 2_pin_Molex_header, J4 3_pin_Molex_header, J5 2_pin_Molex_header, J6 2_pin_Molex_header, Q1 2N3904, Q2 2N3904, SW2 SW_DP3T, U1 TL072, U3 AS3340A, U4 LM4040BIZ-5, U5 LM4040BIZ-5, U6 L79L05_TO92, U7 TL074

Commit message: Revised layout
Parts:
- moved GRAF4 102.8 mm to (168.2, 39.7), turned to 0 degrees
- moved TP2 37.9 mm to (97.8, 77.3)
- moved R27 31.3 mm to (116.9, 53.1), turned to 180 degrees
- moved R31 31.3 mm to (116.9, 49.3), turned to 180 degrees
- moved TP4 28.1 mm to (97.8, 72.2)
- moved R2 19.2 mm to (134.6, 67.1)
- moved J4 18.9 mm to (99.1, 49.3), turned to -90 degrees
- moved J3 16.9 mm to (127.0, 116.0)
- moved J1 13.4 mm to (99.1, 59.5)
- moved R5 12.5 mm to (148.6, 83.6)
- moved R11 12.5 mm to (148.6, 67.1)
- moved R14 11.6 mm to (158.8, 76.0)
- moved R4 11.6 mm to (106.7, 62.0)
- moved R6 11.6 mm to (116.9, 65.8)
- moved R7 11.6 mm to (116.9, 58.2)
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Connections:
- J4 pad 1: /Main PCB/+2V_REF -> /Main PCB/-2V_REF
- J4 pad 3: /Main PCB/-2V_REF -> /Main PCB/+2V_REF
Routing:
- net PWMIN: track 109.7 -> 77.8 mm
- net CV_NODE: track 114.5 -> 87.1 mm
- net Net-(R2-Pad1): track 42.2 -> 14.8 mm
- net Net-(R2-Pad2): track 8.87 -> 29.5 mm
- net /Main PCB/OCTAVE: track 12.0 -> 28.3 mm
- net +5V_REF: track 204.4 -> 189.5 mm
- net V_OCT: track 10.7 -> 21.8 mm
- net +12V: track 244.7 -> 234.4 mm
- net HFT: track 60.8 -> 50.8 mm
- net SIN: track 77.7 -> 67.9 mm
- net -5V: track 104.7 -> 95.0 mm
- net /Main PCB/LIN_FM_IN: track 10.5 -> 19.4 mm
- net PWM_IN: track 71.8 -> 63.2 mm
- net /Main PCB/HI_FREQ_TRACK: track 13.3 -> 21.6 mm
- net /Main PCB/LINK_IN_CV: track 39.7 -> 32.1 mm
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Other:
- outline, holes or cut-outs redrawn
- board text added: "+5V"
- board text added: "-5V"
- board text added: "Fine tune"
- board text added: "HS/Sin/SSoff/SS"
- board text added: "Lin FM in"
- board text added: "Oct"
- board text added: "Saw out"
- board text added: "Tri out"
- board text removed: "Octave"

Commit message: Pre prototype revisions, README revision
Parts:
- R1: renamed from R27; value 300k -> 30k
- R2: renamed from R31; value 300k -> 30k
- moved C10 2.62 mm to (161.4, 87.4)
- moved C11 2.62 mm to (161.4, 98.8)
- moved R12 2.62 mm to (151.2, 95.0)
- moved R14 2.62 mm to (151.2, 67.1)
- moved R16 2.62 mm to (161.4, 76.0)
- moved R17 2.62 mm to (151.2, 91.2)
- moved R18 2.62 mm to (151.2, 79.8)
- moved R19 2.62 mm to (151.2, 63.3)
- moved R28 2.62 mm to (161.4, 72.2)
- moved R9 2.62 mm to (151.2, 83.6)
- moved GRAF2 2.49 mm to (135.7, 188.0)
- moved B2 1.56 mm to (20.0, 106.0)
- moved TP1 1.27 mm to (97.8, 76.0)
- moved TP2 1.27 mm to (97.8, 70.9)
- renumbered C11 to C10, C12 to C11, C13 to C12, C14 to C13, C15 to C14, C16 to C15, C17 to C16, C18 to C17, C19 to C18, C10 to C4, C20 to C5, GRAF2 to GRAF1, GRAF3 to GRAF2, GRAF4 to GRAF3, GRAF1 to GRAF4, J17 to J1, J16 to J14, J19 to J15, J20 to J16, J21 to J17, J22 to J19, J1 to J2, J23 to J20, J24 to J21, J26 to J22, J4 to J3, J2 to J4, J3 to J5, J5 to J6, J6 to J7, R6 to R10, R7 to R11, R18 to R12, R10 to R13, R11 to R14, R13 to R15, R14 to R16, R15 to R17, R19 to R18, R20 to R19, R16 to R20, R17 to R21, R28 to R27, R29 to R28, R30 to R29, R1 to R3, R42 to R34, R43 to R35, R44 to R36, R45 to R37, R46 to R38, R47 to R39, R2 to R4, R48 to R40, R49 to R41, R50 to R42, R51 to R43, R52 to R44, R53 to R45, R54 to R46, R55 to R47, R56 to R48, R57 to R49, R3 to R5, R58 to R50, R59 to R51, R60 to R52, R61 to R53, R62 to R54, R63 to R55, R64 to R56, R65 to R57, R66 to R58, R67 to R59, R8 to R6, R9 to R7, R4 to R8, R5 to R9, RV2 to RV1, RV5 to RV2, RV6 to RV3, RV9 to RV4, RV10 to RV6, RV11 to RV7, RV12 to RV8, TP2 to TP1, TP4 to TP2, TP6 to TP3, TP7 to TP4, TP8 to TP5, TP9 to TP6, U3 to U2, U4 to U3, U5 to U4, U6 to U5, U7 to U6
Routing:
- net LIN_FM: track 41.1 -> 44.3 mm
- net Net-(C4-Pad1): track 16.7 -> 19.5 mm
- net /Main PCB/SOFT_SYNC_OFF: track 12.2 -> 14.8 mm
- net /Main PCB/CENTER_FREQ: track 17.5 -> 14.9 mm
- net /Main PCB/HI_FREQ_TRACK: track 21.6 -> 19.0 mm
- net +12V: track 234.4 -> 237.0 mm
- net Net-(C8-Pad1): track 16.1 -> 18.7 mm
- net -5V: track 95.0 -> 97.2 mm
- net CV_NODE: track 87.1 -> 88.9 mm
- net Net-(R28-Pad1): track 46.5 -> 45.0 mm
- net -5V_REF: track 50.2 -> 49.0 mm
- net +5V_REF: track 189.5 -> 188.2 mm
Other:
- board text added: "Rich Holmes CC0 1.0 / Mar 2022 https://github.com/holmesrichards/sidekick"
- board text removed: "Rich Holmes CC0 1.0 Jan 2022 https://github.com/holmesrichards/sidekick"

Commit message: Fix nuked footprints; update trimmer footprints
Parts:
- RV1, RV2, RV3: footprint Potentiometer_THT:Potentiometer_Bourns_3296P_Horizontal -> ao_tht:Potentiometer_Bourns_3296P_Horizontal
- RV4: value 10k -> 50k; footprint Potentiometer_THT:Potentiometer_Bourns_3296P_Horizontal -> ao_tht:Potentiometer_Bourns_3296P_Horizontal
- SW2: footprint herovco:SW_CK_OS203012MU5QP1_DP3T -> sidekickvco:SW_CK_OS203012MU5QP1_DP3T

Commit message: Matching notes on silk
Other:
- board text added: "Match R8-R10 Match R1-R2 with octave switch"
- board text added: "Match with R8/10"
- board text added: "Match with R9"
- board text added: "Match with oct switch"
Changed lines of the file:
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@@
     (property "Vendor" "Tayda")
     (attr through_hole)
-    (fp_text reference "R10" (at -2.159 0.127) (layer "F.SilkS")
+    (fp_text reference "R10" (at -2.112 0) (layer "F.SilkS")
       (effects (font (size 0.75 0.75) (thickness 0.15)))
     )
@@
     (property "Vendor" "Tayda")
     (attr through_hole)
-    (fp_text reference "C5" (at 2.5 2.286) (layer "F.SilkS")
+    (fp_text reference "C5" (at 7.5 0) (layer "F.SilkS")
       (effects (font (size 0.75 0.75) (thickness 0.15)))
     )
@@
       (net 2 "-5V") (pinfunction "1") (pintype "passive"))
   )
+  (gr_line (start 124.052 44.24) (end 149.452 44.24) (layer "F.SilkS") (width 0.2))
+  (gr_rect (start 105.129 60.115) (end 120.115 70.021) (layer "F.SilkS") (width 0.12) (fill none))
+  (gr_line (start 152.5 55.416) (end 152.5 50.336) (layer "F.SilkS") (width 0.2))
+  (gr_line (start 150.3 87) (end 150.3 85.5205) (layer "F.SilkS") (width 0.12))
   (gr_rect (start 126.338 37.382) (end 173.963 43.478) (layer "F.SilkS") (width 0.12) (fill none))
+  (gr_rect (start 105.1036 47.288) (end 120.115 56.559) (layer "F.SilkS") (width 0.12) (fill none))
+  (gr_line (start 121.004 46.272) (end 121.004 47.288) (layer "F.SilkS") (width 0.2))
+  (gr_line (start 149.452 44.24) (end 150.976 45.764) (layer "F.SilkS") (width 0.2))
+  (gr_line (start 121.004 64.56) (end 143.356 64.56) (layer "F.SilkS") (width 0.2))
+  (gr_line (start 148.944 81.324) (end 148.944 58.972) (layer "F.SilkS") (width 0.2))
+  (gr_line (start 147.928 80.308) (end 148.944 81.324) (layer "F.SilkS") (width 0.2))
+  (gr_line (start 121.004 64.56) (end 122.02 65.576) (layer "F.SilkS") (width 0.2))
+  (gr_line (start 122.02 63.544) (end 121.004 64.56) (layer "F.SilkS") (width 0.2))
+  (gr_line (start 144.499 81.578) (end 144.499 87) (layer "F.SilkS") (width 0.12))
+  (gr_line (start 150.3 85.515) (end 164.946 85.515) (layer "F.SilkS") (width 0.12))
+  (gr_line (start 164.946 85.515) (end 164.946 81.578) (layer "F.SilkS") (width 0.12))
+  (gr_line (start 121.004 47.288) (end 122.02 47.288) (layer "F.SilkS") (width 0.2))
+  (gr_line (start 143.356 64.56) (end 152.5 55.416) (layer "F.SilkS") (width 0.2))
+  (gr_line (start 124.052 44.24) (end 121.004 47.288) (layer "F.SilkS") (width 0.2))
+  (gr_rect (start 150.976 45.256) (end 165.708 50.336) (layer "F.SilkS") (width 0.2) (fill none))
+  (gr_line (start 164.946 81.578) (end 144.499 81.578) (layer "F.SilkS") (width 0.12))
+  (gr_line (start 144.499 87) (end 150.3 87) (layer "F.SilkS") (width 0.12))
+  (gr_line (start 149.96 80.308) (end 148.944 81.324) (layer "F.SilkS") (width 0.2))
   (gr_line (start 76.3 25) (end 76.3 33) (layer "Dwgs.User") (width 0.1))
   (gr_line (start 72.3 29) (end 80.3 29) (layer "Dwgs.User") (width 0.1))
@@
     (effects (font (size 1 1) (thickness 0.15)))
   )
-  (gr_text "+2V" (at 102.97 54.4) (layer "F.SilkS")
+  (gr_text "Match with oct switch\n" (at 112.622 55.67) (layer "F.SilkS")
+    (effects (font (size 1 0.8) (thickness 0.15)))
+  )
+  (gr_text "+2V" (at 102.3604 54.5016) (layer "F.SilkS")
     (effects (font (size 0.75 0.75) (thickness 0.15)) (justify left))
   )
-  (gr_text "-5V" (at 104.113 59.607) (layer "F.SilkS")
+  (gr_text "-5V" (at 103.478 59.607) (layer "F.SilkS")
     (effects (font (size 0.75 0.75) (thickness 0.15)))
   )
@@
     (effects (font (size 1 1) (thickness 0.15)))
   )
+  (gr_text "Match\nwith\nR8/10" (at 144.88 84.372) (layer "F.SilkS")
+    (effects (font (size 1 1) (thickness 0.15)) (justify left))
+  )
+  (gr_text "Match R8-R10\nMatch R1-R2 with\noctave switch" (at 158.2404 47.9484) (layer "F.SilkS")
+    (effects (font (size 1 1) (thickness 0.15)))
+  )
   (gr_text "SS" (at 29.31 110.915 90) (layer "F.SilkS")
     (effects (font (size 1 1) (thickness 0.15)) (justify right))
   )
-  (gr_text "Fine\ntune" (at 104.24 62.02) (layer "F.SilkS")
+  (gr_text "Fine\ntune" (at 103.605 62.02) (layer "F.SilkS")
     (effects (font (size 0.75 0.75) (thickness 0.15)))
   )
+  (gr_text "Match with R9" (at 112.368 68.624) (layer "F.SilkS")
+    (effects (font (size 1 1) (thickness 0.15)))
+  )
   (gr_text "HS" (at 17.88 110.915 90) (layer "F.SilkS")
     (effects (font (size 1 1) (thickness 0.15)) (justify right))
@@
     (effects (font (size 1 1) (thickness 0.15)))
   )
-  (gr_text "-2V" (at 102.97 49.32) (layer "F.SilkS")
+  (gr_text "-2V" (at 102.3604 49.4216) (layer "F.SilkS")
     (effects (font (size 0.75 0.75) (thickness 0.15)) (justify left))
   )
-  (gr_text "Oct" (at 102.97 51.86) (layer "F.SilkS")
+  (gr_text "Oct" (at 102.3604 51.9616) (layer "F.SilkS")
     (effects (font (size 0.75 0.75) (thickness 0.15)) (justify left))
   )
@@
     (effects (font (size 1 1) (thickness 0.15)))
   )
-  (gr_text "+5V" (at 103.986 64.56) (layer "F.SilkS")
+  (gr_text "+5V" (at 103.351 64.56) (layer "F.SilkS")
     (effects (font (size 0.75 0.75) (thickness 0.15)))
   )

Commit message: Less ridiculous routing
Parts:
- moved R23 66.0 mm to (134.7, 46.8)
- moved U3 8.97 mm to (114.4, 40.8)
- moved U4 8.81 mm to (105.5, 40.8)
- moved C4 3.81 mm to (146.1, 109.0)
- moved R25 3.81 mm to (144.8, 58.2)
- moved R26 3.81 mm to (134.6, 62.0)
- moved R29 3.81 mm to (144.8, 50.6)
- moved R27 3.81 mm to (134.6, 54.4)
- moved R6 3.81 mm to (135.9, 112.8)
Routing:
- net +5V_REF: track 188.2 -> 109.0 mm
- net Net-(R25-Pad1): track 21.7 -> 31.8 mm
- net +12V: track 237.0 -> 242.2 mm
- net /Main PCB/LINK_IN_PW: track 63.7 -> 59.2 mm
- net PWMIN: track 77.8 -> 73.9 mm
- net Net-(R28-Pad1): track 45.0 -> 41.2 mm
- net Net-(C4-Pad1): track 19.5 -> 21.9 mm
- net -5V_REF: track 49.0 -> 47.5 mm
- net Net-(R27-Pad1): track 9.95 -> 9.41 mm
- net /Main PCB/LIN_FM_IN: track 19.4 -> 18.9 mm
