File: Hardware/PCB/sidekickvco/sidekickvco.kicad_pcb (KiCad board)
At the start: 2 copper layers, 169.5 x 163 mm, 123 parts, among them J1 Conn_02x04_Odd_Even, J14 Wire pad, J15 Wire pad, J16 Wire pad, J17 Wire pad, J18 AudioJack2, J19 AudioJack2, J2 3_pin_Molex_header, J20 Synth_power_2x5, J21 AudioJack2, J22 AudioJack2, J3 3_pin_Molex_header, J4 4_pin_Molex_header, J5 2_pin_Molex_header, J6 2_pin_Molex_header, J7 2_pin_Molex_header, Q1 2N3904, Q2 2N3904, SW2 SW_DP3T, U1 TL072, U2 AS3340A, U3 LM4040BIZ-5, U4 LM4040BIZ-5, U5 L79L05_TO92, U6 TL074

Commit message: More routing tweaks
Routing:
- net /Main PCB/LIN_FM_IN: track 18.9 -> 17.8 mm
- net SAW_OUT: track 78.7 -> 78.0 mm
Changed lines of the file:
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@@
   (segment (start 130.83 98.85) (end 135.91 98.85) (width 0.25) (layer "B.Cu") (net 33))
   (segment (start 135.91 98.85) (end 137.18 97.58) (width 0.25) (layer "B.Cu") (net 33))
-  (segment (start 144.8 111.55) (end 146.07 112.82) (width 0.25) (layer "B.Cu") (net 34))
-  (segment (start 130.68 115.995) (end 135.125 111.55) (width 0.25) (layer "B.Cu") (net 34))
-  (segment (start 135.125 111.55) (end 144.8 111.55) (width 0.25) (layer "B.Cu") (net 34))
-  (segment (start 129.56 115.995) (end 130.68 115.995) (width 0.25) (layer "B.Cu") (net 34))
+  (segment (start 144.927 113.963) (end 146.07 112.82) (width 0.25) (layer "B.Cu") (net 34))
+  (segment (start 129.56 115.995) (end 131.592 113.963) (width 0.25) (layer "B.Cu") (net 34))
+  (segment (start 131.592 113.963) (end 144.927 113.963) (width 0.25) (layer "B.Cu") (net 34))
   (segment (start 99.14 49.32) (end 106.78 49.32) (width 0.25) (layer "B.Cu") (net 35))
   (segment (start 122.650311 51.86) (end 123.46452 52.674209) (width 0.25) (layer "B.Cu") (net 36))
@@
   (segment (start 121.95 89.96) (end 123.21 91.22) (width 0.25) (layer "F.Cu") (net 56))
   (via (at 123.21 110.026) (size 0.8) (drill 0.4) (layers "F.Cu" "B.Cu") (net 56))
-  (segment (start 123.21 120.44) (end 123.21 110.026) (width 0.25) (layer "B.Cu") (net 56))
+  (segment (start 123.21 119.17) (end 123.21 110.026) (width 0.25) (layer "B.Cu") (net 56))
+  (segment (start 147.721 127.494996) (end 146.711983 126.485979) (width 0.25) (layer "B.Cu") (net 56))
   (segment (start 147.721 145.449) (end 147.721 127.494996) (width 0.25) (layer "B.Cu") (net 56))
-  (segment (start 130.525979 126.485979) (end 124.48 120.44) (width 0.25) (layer "B.Cu") (net 56))
-  (segment (start 124.48 120.44) (end 123.21 120.44) (width 0.25) (layer "B.Cu") (net 56))
+  (segment (start 146.06 147.11) (end 147.721 145.449) (width 0.25) (layer "B.Cu") (net 56))
   (segment (start 146.711983 126.485979) (end 130.525979 126.485979) (width 0.25) (layer "B.Cu") (net 56))
-  (segment (start 147.721 127.494996) (end 146.711983 126.485979) (width 0.25) (layer "B.Cu") (net 56))
-  (segment (start 146.06 147.11) (end 147.721 145.449) (width 0.25) (layer "B.Cu") (net 56))
+  (segment (start 130.525979 126.485979) (end 123.21 119.17) (width 0.25) (layer "B.Cu") (net 56))
   (segment (start 105.43 143.31) (end 106.554511 142.185489) (width 0.25) (layer "F.Cu") (net 57))
   (segment (start 106.554511 142.185489) (end 106.554511 135.544511) (width 0.25) (layer "F.Cu") (net 57))

Commit message: Adjust trimmer footprints
Parts:
- moved RV1 1.00 mm to (172.3, 72.0)
- moved RV2 1.00 mm to (172.3, 96.0)
- moved RV3 1.00 mm to (172.3, 60.0)
- moved RV4 1.00 mm to (172.3, 84.0)
Routing:
- net /Main PCB/HI_FREQ_TRACK: track 19.0 -> 20.0 mm
- net PWM_IN: track 63.2 -> 64.2 mm
- net Net-(R4-Pad2): track 29.5 -> 30.5 mm
- net Net-(R28-Pad1): track 41.2 -> 42.2 mm
- net HFT: track 50.8 -> 51.8 mm
- net /Main PCB/CENTER_FREQ: track 14.9 -> 15.9 mm
- net -5V: track 97.2 -> 98.2 mm
- net +5V_REF: track 109.0 -> 110.0 mm

Commit message: Fix lin FM input, add howitworks
Parts:
- removed R7: 100k, ao_tht:R_Axial_DIN0207_L6.3mm_D2.5mm_P10.16mm_Horizontal
Connections:
- C4 pad 2: Net-(C4-Pad2) -> /Main PCB/LIN_FM_IN
- C5 pad 2: Net-(C5-Pad2) -> /Main PCB/LINK_IN_FM
- R6 pad 1: Net-(C4-Pad2) -> /Main PCB/LIN_FM_IN
- R6 pad 2: /Main PCB/LIN_FM_IN -> GND
Routing:
- net /Main PCB/LINK_IN_FM: track 31.3 -> 43.5 mm, vias 0 -> 1
- net Net-(C5-Pad2): track 11.0 -> 0.00 mm
- net Net-(C4-Pad2): track 6.74 -> 0.00 mm
- net /Main PCB/LIN_FM_IN: track 17.8 -> 14.4 mm

Commit message: Restore resistor
Parts:
- added R7: 100k, ao_tht:R_Axial_DIN0207_L6.3mm_D2.5mm_P10.16mm_Horizontal, F.Cu at (115.7, 72.2)
Routing:
- net /Main PCB/LINK_IN_FM: vias 1 -> 0
Changed lines of the file:
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@@
+  )
+  (footprint "ao_tht:R_Axial_DIN0207_L6.3mm_D2.5mm_P10.16mm_Horizontal" (layer "F.Cu")
+    (at 115.67 72.18 180)
+    (descr "Resistor, Axial_DIN0207 series, Axial, Horizontal, pin pitch=10.16mm, 0.25W = 1/4W, length*diameter=6.3*2.5mm^2, http://cdn-reichelt.de/documents/datenblatt/B400/1_4W%23YAG.pdf")
+    (tags "Resistor Axial_DIN0207 series Axial Horizontal pin pitch 10.16mm 0.25W = 1/4W length 6.3mm diameter 2.5mm")
+    (property "Sheetfile" "sidekickvco_main.kicad_sch")
+    (property "Sheetname" "Main PCB")
+    (property "Vendor" "Tayda")
+    (attr through_hole)
+    (fp_text reference "R7" (at 5.08 -2.37) (layer "F.SilkS")
+      (effects (font (size 0.75 0.75) (thickness 0.15)))
+    )
+    (fp_text value "100k" (at 5.08 2.37) (layer "F.Fab")
+      (effects (font (size 1 1) (thickness 0.15)))
+    )
+    (fp_text user "${VALUE}" (at 5.08 0) (layer "F.SilkS")
+      (effects (font (size 0.75 0.75) (thickness 0.15)))
+    )
+    (fp_text user "${REFERENCE}" (at 5.08 0) (layer "F.Fab")
+      (effects (font (size 1 1) (thickness 0.15)))
+    )
+    (fp_line (start 1.81 -1.37) (end 1.81 1.37) (layer "F.SilkS") (width 0.12))
+    (fp_line (start 8.35 -1.37) (end 1.81 -1.37) (layer "F.SilkS") (width 0.12))
+    (fp_line (start 8.35 1.37) (end 8.35 -1.37) (layer "F.SilkS") (width 0.12))
+    (fp_line (start 1.81 1.37) (end 8.35 1.37) (layer "F.SilkS") (width 0.12))
+    (fp_line (start 1.04 0) (end 1.81 0) (layer "F.SilkS") (width 0.12))
+    (fp_line (start 9.12 0) (end 8.35 0) (layer "F.SilkS") (width 0.12))
+    (fp_line (start -1.05 -1.5) (end -1.05 1.5) (layer "F.CrtYd") (width 0.05))
+    (fp_line (start 11.21 1.5) (end 11.21 -1.5) (layer "F.CrtYd") (width 0.05))
+    (fp_line (start 11.21 -1.5) (end -1.05 -1.5) (layer "F.CrtYd") (width 0.05))
+    (fp_line (start -1.05 1.5) (end 11.21 1.5) (layer "F.CrtYd") (width 0.05))
+    (fp_line (start 8.23 -1.25) (end 1.93 -1.25) (layer "F.Fab") (width 0.1))
+    (fp_line (start 1.93 -1.25) (end 1.93 1.25) (layer "F.Fab") (width 0.1))
+    (fp_line (start 8.23 1.25) (end 8.23 -1.25) (layer "F.Fab") (width 0.1))
+    (fp_line (start 10.16 0) (end 8.23 0) (layer "F.Fab") (width 0.1))
+    (fp_line (start 1.93 1.25) (end 8.23 1.25) (layer "F.Fab") (width 0.1))
+    (fp_line (start 0 0) (end 1.93 0) (layer "F.Fab") (width 0.1))
+    (pad "1" thru_hole circle locked (at 0 0 180) (size 1.6 1.6) (drill 0.8) (layers *.Cu *.Mask)
+      (net 41 "/Main PCB/LINK_IN_FM") (pintype "passive"))
+    (pad "2" thru_hole oval locked (at 10.16 0 180) (size 1.6 1.6) (drill 0.8) (layers *.Cu *.Mask)
+      (net 1 "GND") (pintype "passive"))
+    (model "${KICAD_AOKICAD}/ao_tht_3d/R_Axial_DIN0207_L6.3mm_D2.5mm_P10.16mm_Horizontal.wrl"
+      (offset (xyz 0 0 0))
+      (scale (xyz 1 1 1))
+      (rotate (xyz 0 0 0))
+    )
   )
   (footprint "ao_tht:R_Axial_DIN0207_L6.3mm_D2.5mm_P10.16mm_Horizontal" (layer "F.Cu")
@@
   (segment (start 110.717 94.103282) (end 112.134031 95.520313) (width 0.25) (layer "F.Cu") (net 41))
   (segment (start 115.59 72.18) (end 110.705489 77.064511) (width 0.25) (layer "F.Cu") (net 41))
-  (via (at 115.59 72.18) (size 0.8) (drill 0.4) (layers "F.Cu" "B.Cu") (net 41))
   (segment (start 119.44 72.18) (end 124.52 67.1) (width 0.25) (layer "B.Cu") (net 41))
   (segment (start 115.59 72.18) (end 119.44 72.18) (width 0.25) (layer "B.Cu") (net 41))
