File: Hardware/PCB/sidekickvco/sidekickvco.kicad_sch (KiCad schematic)
At the start: 17 parts, among them J1 Conn_02x04_Odd_Even, J10 4_pin_Molex_connector, J11 2_pin_Molex_connector, J12 2_pin_Molex_connector, J13 2_pin_Molex_connector, J14 Wire pad, J15 Wire pad, J16 Wire pad, J17 Wire pad, J2 3_pin_Molex_header, J3 3_pin_Molex_header, J4 4_pin_Molex_header, J5 2_pin_Molex_header, J6 2_pin_Molex_header, J7 2_pin_Molex_header, J8 3_pin_Molex_connector, J9 3_pin_Molex_connector

Commit message: BOM
Parts:
- J14: value Wire pad -> (none); footprint Connector_Wire:SolderWire-0.5sqmm_1x01_D0.9mm_OD2.1mm -> (none); now left out of the parts list
- J15, J16, J17: value Wire pad -> (none); footprint sidekickvco:SolderWire-round_1x01_D0.9mm_OD2.1mm -> (none); now left out of the parts list
Changed lines of the file:
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@@
   )
   (symbol (lib_id "Connector_Generic:Conn_01x01") (at 160.02 96.52 0) (unit 1)
-    (in_bom yes) (on_board yes)
+    (in_bom no) (on_board yes)
     (property "Reference" "J14" (id 0) (at 162.052 95.6115 0)
       (effects (font (size 1.27 1.27)) (justify left))
     )
-    (property "Value" "Wire pad" (id 1) (at 154.94 106.68 0)
+    (property "Value" "" (id 1) (at 154.94 106.68 0)
       (effects (font (size 1.27 1.27)) (justify left))
     )
-    (property "Footprint" "Connector_Wire:SolderWire-0.5sqmm_1x01_D0.9mm_OD2.1mm" (id 2) (at 160.02 96.52 0)
+    (property "Footprint" "" (id 2) (at 160.02 96.52 0)
       (effects (font (size 1.27 1.27)) hide)
     )
@@
   )
   (symbol (lib_id "Connector_Generic:Conn_01x01") (at 160.02 99.06 0) (unit 1)
-    (in_bom yes) (on_board yes) (fields_autoplaced)
+    (in_bom no) (on_board yes) (fields_autoplaced)
     (property "Reference" "J15" (id 0) (at 162.052 98.1515 0)
       (effects (font (size 1.27 1.27)) (justify left))
     )
-    (property "Value" "Wire pad" (id 1) (at 162.052 100.9266 0)
+    (property "Value" "" (id 1) (at 162.052 100.9266 0)
       (effects (font (size 1.27 1.27)) (justify left) hide)
     )
-    (property "Footprint" "sidekickvco:SolderWire-round_1x01_D0.9mm_OD2.1mm" (id 2) (at 160.02 99.06 0)
+    (property "Footprint" "" (id 2) (at 160.02 99.06 0)
       (effects (font (size 1.27 1.27)) hide)
     )
@@
   )
   (symbol (lib_id "Connector_Generic:Conn_01x01") (at 160.02 101.6 0) (unit 1)
-    (in_bom yes) (on_board yes) (fields_autoplaced)
+    (in_bom no) (on_board yes) (fields_autoplaced)
     (property "Reference" "J16" (id 0) (at 162.052 100.6915 0)
       (effects (font (size 1.27 1.27)) (justify left))
     )
-    (property "Value" "Wire pad" (id 1) (at 162.052 103.4666 0)
+    (property "Value" "" (id 1) (at 162.052 103.4666 0)
       (effects (font (size 1.27 1.27)) (justify left) hide)
     )
-    (property "Footprint" "sidekickvco:SolderWire-round_1x01_D0.9mm_OD2.1mm" (id 2) (at 160.02 101.6 0)
+    (property "Footprint" "" (id 2) (at 160.02 101.6 0)
       (effects (font (size 1.27 1.27)) hide)
     )
@@
   )
   (symbol (lib_id "Connector_Generic:Conn_01x01") (at 160.02 104.14 0) (unit 1)
-    (in_bom yes) (on_board yes) (fields_autoplaced)
+    (in_bom no) (on_board yes) (fields_autoplaced)
     (property "Reference" "J17" (id 0) (at 162.052 103.2315 0)
       (effects (font (size 1.27 1.27)) (justify left))
     )
-    (property "Value" "Wire pad" (id 1) (at 162.052 106.0066 0)
+    (property "Value" "" (id 1) (at 162.052 106.0066 0)
       (effects (font (size 1.27 1.27)) (justify left) hide)
     )
-    (property "Footprint" "sidekickvco:SolderWire-round_1x01_D0.9mm_OD2.1mm" (id 2) (at 160.02 104.14 0)
+    (property "Footprint" "" (id 2) (at 160.02 104.14 0)
       (effects (font (size 1.27 1.27)) hide)
     )
