File: Hardware/PCB/sidekickvco/sidekickvco.kicad_sch (KiCad schematic)
At the start: 17 parts, among them J1 Conn_02x04_Odd_Even, J10 4_pin_Molex_connector, J11 2_pin_Molex_connector, J12 2_pin_Molex_connector, J13 2_pin_Molex_connector, J2 3_pin_Molex_header, J3 3_pin_Molex_header, J4 4_pin_Molex_header, J5 2_pin_Molex_header, J6 2_pin_Molex_header, J7 2_pin_Molex_header, J8 3_pin_Molex_connector, J9 3_pin_Molex_connector

Commit message: Fix nuked footprints; update trimmer footprints
Parts:
- J1: value Conn_02x04_Odd_Even -> (none); footprint Connector_IDC:IDC-Header_2x04_P2.54mm_Vertical -> (none)
- J10: value 4_pin_Molex_connector -> (none)
- J11, J12, J13: value 2_pin_Molex_connector -> (none)
- J2, J3: value 3_pin_Molex_header -> (none); footprint ao_tht:Molex_KK-254_AE-6410-03A_1x03_P2.54mm_Vertical -> (none)
- J4: value 4_pin_Molex_header -> (none); footprint Connector_Molex:Molex_KK-254_AE-6410-04A_1x04_P2.54mm_Vertical -> (none)
- J5, J6, J7: value 2_pin_Molex_header -> (none); footprint ao_tht:Molex_KK-254_AE-6410-02A_1x02_P2.54mm_Vertical -> (none)
- J8, J9: value 3_pin_Molex_connector -> (none); footprint ao_tht:Molex_KK-254_AE-6410-03A_1x03_P2.54mm_Vertical -> (none)

Commit message: Post prototype updates
Parts:
- J1: value (none) -> Conn_02x04_Odd_Even; footprint (none) -> Connector_IDC:IDC-Header_2x04_P2.54mm_Vertical; SKU (none) -> A-2948; Vendor (none) -> Tayda
- J10: value (none) -> 4_pin_Molex_connector; SKU (none) -> A-828; Vendor (none) -> Tayda
- J11, J12, J13: value (none) -> 2_pin_Molex_connector
- J14: value (none) -> Wire pad; footprint (none) -> Connector_Wire:SolderWire-0.5sqmm_1x01_D0.9mm_OD2.1mm
- J15, J16, J17: value (none) -> Wire pad; footprint (none) -> sidekickvco:SolderWire-round_1x01_D0.9mm_OD2.1mm
- J2, J3: value (none) -> 3_pin_Molex_header; footprint (none) -> ao_tht:Molex_KK-254_AE-6410-03A_1x03_P2.54mm_Vertical
- J4: value (none) -> 4_pin_Molex_header; footprint (none) -> Connector_Molex:Molex_KK-254_AE-6410-04A_1x04_P2.54mm_Vertical; SKU (none) -> A-806; Vendor (none) -> Tayda
- J5, J6, J7: value (none) -> 2_pin_Molex_header; footprint (none) -> ao_tht:Molex_KK-254_AE-6410-02A_1x02_P2.54mm_Vertical
- J8, J9: value (none) -> 3_pin_Molex_connector; footprint (none) -> ao_tht:Molex_KK-254_AE-6410-03A_1x03_P2.54mm_Vertical
