File: Hardware/PCB/sidekickvco/panel.kicad_sch (KiCad schematic)
At the start: 7 parts, among them SW1 SW_Rotary12, SW2 SW_DP3T

Commit message: Initial version of circuit and layout
Parts:
- added J13, J14, J15: AudioJack2, ao_tht:Jack_6.35mm_PJ_629HAN, symbol ao_symbols:AudioJack2
- added RV1: 100k, ao_tht:Potentiometer_Alpha_RD901F-40-00D_Single_Vertical_centered, symbol ao_symbols:R_POT
Connections:
- new net +5VREF_P: RV1.3
- new net -5VREF_P: RV1.1
- new net FINE_TUNE_P: RV1.2
- new net GND1: J13.S, J14.S, J15.S
- new net LIN_FM_IN_J: J13.T
- new net SAW_P: J15.T
- new net TRI_P: J14.T
Other:
- note added: "JACKS"
- note added: "POT"
- moved on the sheet: B3, R35, R36, R37, R38, SW1, SW2A, SW2B

Commit message: Daughterboard mounting
Parts:
- added GRAF1: board, sidekickvco:sidekick_daughterboard, symbol ao_symbols:Graphic
- added H1, H2: MountingHole, ao_tht:MountingHole_3.2mm_M3, symbol ao_symbols:MountingHole
Other:
- note removed: "Panel mounted"
- moved on the sheet: B3
Changed lines of the file:
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@@
     (stroke (width 0) (type default) (color 0 0 0 0))
-  )
-  (text "Panel mounted" (at 110.49 41.91 0)
-    (effects (font (size 1.27 1.27)) (justify left bottom))
   )
   (text "SYNC\nSWITCH" (at 162.56 36.83 0)
@@
   )
   (text "Precision or hand matched resistors" (at 67.31 89.535 0)
-    (effects (font (size 1.27 1.27)) (justify left bottom))
-  )
-  (text "Panel mounted" (at 167.64 48.26 0)
     (effects (font (size 1.27 1.27)) (justify left bottom))
   )
@@
     (pin "2")
   )
+  (symbol (lib_id "ao_symbols:Graphic") (at 201.93 38.1 0) (unit 1)
+    (in_bom yes) (on_board yes) (fields_autoplaced)
+    (property "Reference" "GRAF1" (id 0) (at 208.915 37.1915 0)
+      (effects (font (size 1.27 1.27)) (justify left))
+    )
+    (property "Value" "board" (id 1) (at 208.915 39.9666 0)
+      (effects (font (size 1.27 1.27)) (justify left))
+    )
+    (property "Footprint" "sidekickvco:sidekick_daughterboard" (id 2) (at 201.93 38.1 0)
+      (effects (font (size 1.27 1.27)) hide)
+    )
+    (property "Datasheet" "" (id 3) (at 201.93 38.1 0)
+      (effects (font (size 1.27 1.27)) hide)
+    )
+    (property "Config" "DNF" (id 4) (at 201.93 38.1 0)
+      (effects (font (size 1.27 1.27)) hide)
+    )
+  )
   (symbol (lib_id "power:GND1") (at 88.9 147.32 0) (unit 1)
     (in_bom yes) (on_board yes)
@@
     )
     (pin "1")
+  )
+  (symbol (lib_id "ao_symbols:MountingHole") (at 204.47 54.61 0) (unit 1)
+    (in_bom no) (on_board yes) (fields_autoplaced)
+    (property "Reference" "H2" (id 0) (at 207.01 53.7015 0)
+      (effects (font (size 1.27 1.27)) (justify left))
+    )
+    (property "Value" "MountingHole" (id 1) (at 207.01 56.4766 0)
+      (effects (font (size 1.27 1.27)) (justify left))
+    )
+    (property "Footprint" "ao_tht:MountingHole_3.2mm_M3" (id 2) (at 204.47 54.61 0)
+      (effects (font (size 1.27 1.27)) hide)
+    )
+    (property "Datasheet" "" (id 3) (at 204.47 54.61 0)
+      (effects (font (size 1.27 1.27)) hide)
+    )
+    (property "Config" "DNF" (id 4) (at 204.47 54.61 0)
+      (effects (font (size 1.27 1.27)) hide)
+    )
   )
   (symbol (lib_id "ao_symbols:AudioJack2") (at 95.25 143.51 180) (unit 1)
@@
     (pin "4")
   )
+  (symbol (lib_id "ao_symbols:MountingHole") (at 204.47 48.26 0) (unit 1)
+    (in_bom no) (on_board yes) (fields_autoplaced)
+    (property "Reference" "H1" (id 0) (at 207.01 47.3515 0)
+      (effects (font (size 1.27 1.27)) (justify left))
+    )
+    (property "Value" "MountingHole" (id 1) (at 207.01 50.1266 0)
+      (effects (font (size 1.27 1.27)) (justify left))
+    )
+    (property "Footprint" "ao_tht:MountingHole_3.2mm_M3" (id 2) (at 204.47 48.26 0)
+      (effects (font (size 1.27 1.27)) hide)
+    )
+    (property "Datasheet" "" (id 3) (at 204.47 48.26 0)
+      (effects (font (size 1.27 1.27)) hide)
+    )
+    (property "Config" "DNF" (id 4) (at 204.47 48.26 0)
+      (effects (font (size 1.27 1.27)) hide)
+    )
+  )
   (symbol (lib_id "power:GND1") (at 88.9 162.56 0) (unit 1)
     (in_bom yes) (on_board yes)
@@
     (pin "8")
   )
-  (symbol (lib_id "ao_symbols:Board") (at 208.28 41.91 0) (unit 1)
+  (symbol (lib_id "ao_symbols:Board") (at 203.2 27.94 0) (unit 1)
     (in_bom yes) (on_board yes) (fields_autoplaced)
-    (property "Reference" "B3" (id 0) (at 213.995 41.0015 0)
-      (effects (font (size 1.27 1.27)) (justify left))
-    )
-    (property "Value" "Board" (id 1) (at 213.995 43.7766 0)
-      (effects (font (size 1.27 1.27)) (justify left))
-    )
-    (property "Footprint" "ao_tht:Board_Marker" (id 2) (at 208.28 41.91 0)
-      (effects (font (size 1.27 1.27)) hide)
-    )
-    (property "Datasheet" "" (id 3) (at 208.28 41.91 0)
-      (effects (font (size 1.27 1.27)) hide)
-    )
-    (property "Config" "DNF" (id 4) (at 208.28 41.91 0)
-      (effects (font (size 1.27 1.27)) hide)
-    )
+    (property "Reference" "B3" (id 0) (at 208.915 27.0315 0)
+      (effects (font (size 1.27 1.27)) (justify left))
+    )
+    (property "Value" "Board" (id 1) (at 208.915 29.8066 0)
+      (effects (font (size 1.27 1.27)) (justify left))
+    )
+    (property "Footprint" "ao_tht:Board_Marker" (id 2) (at 203.2 27.94 0)
+      (effects (font (size 1.27 1.27)) hide)
+    )
+    (property "Datasheet" "" (id 3) (at 203.2 27.94 0)
+      (effects (font (size 1.27 1.27)) hide)
+    )
+    (property "Config" "DNF" (id 4) (at 203.2 27.94 0)
+      (effects (font (size 1.27 1.27)) hide)
+    )

Commit message: Revise layout, add notes, BUILD.md
Parts:
- renumbered B3 to B2
Changed lines of the file:
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@@
   (symbol (lib_id "ao_symbols:Board") (at 203.2 27.94 0) (unit 1)
     (in_bom yes) (on_board yes) (fields_autoplaced)
-    (property "Reference" "B3" (id 0) (at 208.915 27.0315 0)
+    (property "Reference" "B2" (id 0) (at 208.915 27.0315 0)
       (effects (font (size 1.27 1.27)) (justify left))
     )

Commit message: Correct slide switch footprint; use TO-92 wide for regulator
Connections:
- net HARD_SYNCA_P: now also SW2.5; no longer SW2.1
- net SOFT_SYNCA_P: now also SW2.2, SW2.8; no longer SW2.4, SW2.6
- net SOFT_SYNC_OFF_P: now also SW2.1, SW2.3; no longer SW2.5, SW2.7
- net SYNCA_P: now also SW2.6; no longer SW2.2
Other:
- moved on the sheet: SW2A, SW2B
Changed lines of the file:
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@@
     (pin "T")
   )
-  (symbol (lib_name "SW_DP3T_1") (lib_id "herovco:SW_DP3T") (at 173.99 68.58 0) (unit 1)
+  (symbol (lib_name "SW_DP3T_1") (lib_id "herovco:SW_DP3T") (at 186.69 82.55 0) (unit 1)
     (in_bom yes) (on_board yes) (fields_autoplaced)
-    (property "Reference" "SW2" (id 0) (at 173.99 61.7433 0))
-    (property "Value" "SW_DP3T" (id 1) (at 173.99 64.5184 0))
-    (property "Footprint" "herovco:SW_CK_OS203012MU5QP1_DP3T" (id 2) (at 158.115 64.135 0)
+    (property "Reference" "SW2" (id 0) (at 186.69 75.7133 0))
+    (property "Value" "SW_DP3T" (id 1) (at 186.69 78.4884 0))
+    (property "Footprint" "herovco:SW_CK_OS203012MU5QP1_DP3T" (id 2) (at 170.815 78.105 0)
       (effects (font (size 1.27 1.27)) hide)
     )
-    (property "Datasheet" "~" (id 3) (at 158.115 64.135 0)
+    (property "Datasheet" "~" (id 3) (at 170.815 78.105 0)
       (effects (font (size 1.27 1.27)) hide)
     )
-    (property "Manufacturer" "C&K" (id 4) (at 173.99 68.58 0)
+    (property "Manufacturer" "C&K" (id 4) (at 186.69 82.55 0)
       (effects (font (size 1.27 1.27)) hide)
     )
-    (property "Part" "OS203012MU5QP1‎" (id 5) (at 173.99 68.58 0)
+    (property "Part" "OS203012MU5QP1‎" (id 5) (at 186.69 82.55 0)
       (effects (font (size 1.27 1.27)) hide)
     )
-    (property "Vendor" "Digi-Key" (id 6) (at 173.99 68.58 0)
+    (property "Vendor" "Digi-Key" (id 6) (at 186.69 82.55 0)
       (effects (font (size 1.27 1.27)) hide)
     )
-    (property "SKU" "CKN9554-ND" (id 7) (at 173.99 68.58 0)
+    (property "SKU" "CKN9554-ND" (id 7) (at 186.69 82.55 0)
       (effects (font (size 1.27 1.27)) hide)
     )
@@
     (pin "1")
   )
-  (symbol (lib_id "herovco:SW_DP3T") (at 186.69 82.55 0) (unit 2)
+  (symbol (lib_id "herovco:SW_DP3T") (at 173.99 68.58 0) (unit 2)
     (in_bom yes) (on_board yes) (fields_autoplaced)
-    (property "Reference" "SW2" (id 0) (at 186.69 75.7133 0))
-    (property "Value" "SW_DP3T" (id 1) (at 186.69 78.4884 0))
-    (property "Footprint" "herovco:SW_CK_OS203012MU5QP1_DP3T" (id 2) (at 170.815 78.105 0)
+    (property "Reference" "SW2" (id 0) (at 173.99 61.7433 0))
+    (property "Value" "SW_DP3T" (id 1) (at 173.99 64.5184 0))
+    (property "Footprint" "herovco:SW_CK_OS203012MU5QP1_DP3T" (id 2) (at 158.115 64.135 0)
       (effects (font (size 1.27 1.27)) hide)
     )
-    (property "Datasheet" "~" (id 3) (at 170.815 78.105 0)
+    (property "Datasheet" "~" (id 3) (at 158.115 64.135 0)
       (effects (font (size 1.27 1.27)) hide)
     )
-    (property "Manufacturer" "C&K" (id 4) (at 186.69 82.55 0)
+    (property "Manufacturer" "C&K" (id 4) (at 173.99 68.58 0)
       (effects (font (size 1.27 1.27)) hide)
     )
-    (property "Part" "OS203012MU5QP1‎" (id 5) (at 186.69 82.55 0)
+    (property "Part" "OS203012MU5QP1‎" (id 5) (at 173.99 68.58 0)
       (effects (font (size 1.27 1.27)) hide)
     )
-    (property "Vendor" "Digi-Key" (id 6) (at 186.69 82.55 0)
+    (property "Vendor" "Digi-Key" (id 6) (at 173.99 68.58 0)
       (effects (font (size 1.27 1.27)) hide)
     )
-    (property "SKU" "CKN9554-ND" (id 7) (at 186.69 82.55 0)
+    (property "SKU" "CKN9554-ND" (id 7) (at 173.99 68.58 0)
       (effects (font (size 1.27 1.27)) hide)
     )

Commit message: Pre prototype revisions, README revision
Parts:
- B2: now left out of the parts list
- GRAF4: renamed from GRAF1; now left out of the parts list
- R30: renamed from R35; value 100k 1/8W -> 10k 1/8W
- R31: renamed from R36; value 100k 1/8W -> 10k 1/8W
- R32: renamed from R37; value 100k 1/8W -> 10k 1/8W
- R33: renamed from R38; value 100k 1/8W -> 10k 1/8W
- renumbered J13 to J23, J14 to J24, J15 to J25, RV1 to RV5
Changed lines of the file:
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@@
   (title_block
     (title "Sidekick VCO")
-    (date "2022-01-30")
+    (date "2022-03-12")
     (company "Rich Holmes / Analog Output")
     (comment 1 "or neighboring rights to this work. Published from United States.")
     (comment 2 "To the extent possible under law, Richard Holmes has waived all copyright and related ")
-    (comment 3 "Partly based on designs by Kassutronics, Thomas Henry, and LMNC")
   )
   (junction (at 83.82 72.39) (diameter 0) (color 0 0 0 0)
@@
   (symbol (lib_id "ao_symbols:R") (at 83.82 53.34 0) (mirror x) (unit 1)
     (in_bom yes) (on_board no)
-    (property "Reference" "R35" (id 0) (at 85.09 51.435 0)
-      (effects (font (size 1.27 1.27)) (justify left))
-    )
-    (property "Value" "100k 1/8W" (id 1) (at 85.09 53.34 0)
+    (property "Reference" "R30" (id 0) (at 85.09 51.435 0)
+      (effects (font (size 1.27 1.27)) (justify left))
+    )
+    (property "Value" "10k 1/8W" (id 1) (at 85.09 53.34 0)
       (effects (font (size 1.27 1.27)) (justify left))
     )
@@
   (symbol (lib_id "ao_symbols:R") (at 83.82 60.96 0) (mirror x) (unit 1)
     (in_bom yes) (on_board no)
-    (property "Reference" "R36" (id 0) (at 85.09 59.055 0)
-      (effects (font (size 1.27 1.27)) (justify left))
-    )
-    (property "Value" "100k 1/8W" (id 1) (at 85.09 60.96 0)
+    (property "Reference" "R31" (id 0) (at 85.09 59.055 0)
+      (effects (font (size 1.27 1.27)) (justify left))
+    )
+    (property "Value" "10k 1/8W" (id 1) (at 85.09 60.96 0)
       (effects (font (size 1.27 1.27)) (justify left))
     )
@@
   (symbol (lib_id "ao_symbols:R") (at 83.82 68.58 0) (mirror x) (unit 1)
     (in_bom yes) (on_board no)
-    (property "Reference" "R37" (id 0) (at 85.09 66.675 0)
-      (effects (font (size 1.27 1.27)) (justify left))
-    )
-    (property "Value" "100k 1/8W" (id 1) (at 85.09 68.58 0)
+    (property "Reference" "R32" (id 0) (at 85.09 66.675 0)
+      (effects (font (size 1.27 1.27)) (justify left))
+    )
+    (property "Value" "10k 1/8W" (id 1) (at 85.09 68.58 0)
       (effects (font (size 1.27 1.27)) (justify left))
     )
@@
   (symbol (lib_id "ao_symbols:R") (at 83.82 76.2 0) (mirror x) (unit 1)
     (in_bom yes) (on_board no)
-    (property "Reference" "R38" (id 0) (at 85.09 74.295 0)
-      (effects (font (size 1.27 1.27)) (justify left))
-    )
-    (property "Value" "100k 1/8W" (id 1) (at 85.09 76.2 0)
+    (property "Reference" "R33" (id 0) (at 85.09 74.295 0)
+      (effects (font (size 1.27 1.27)) (justify left))
+    )
+    (property "Value" "10k 1/8W" (id 1) (at 85.09 76.2 0)
       (effects (font (size 1.27 1.27)) (justify left))
     )
@@
   )
   (symbol (lib_id "ao_symbols:Graphic") (at 201.93 38.1 0) (unit 1)
-    (in_bom yes) (on_board yes) (fields_autoplaced)
-    (property "Reference" "GRAF1" (id 0) (at 208.915 37.1915 0)
+    (in_bom no) (on_board yes) (fields_autoplaced)
+    (property "Reference" "GRAF4" (id 0) (at 208.915 37.1915 0)
       (effects (font (size 1.27 1.27)) (justify left))
     )
@@
   (symbol (lib_id "power:GND1") (at 88.9 147.32 0) (unit 1)
     (in_bom yes) (on_board yes)
-    (property "Reference" "#PWR03" (id 0) (at 88.9 153.67 0)
+    (property "Reference" "#PWR045" (id 0) (at 88.9 153.67 0)
       (effects (font (size 1.27 1.27)) hide)
     )
@@
   (symbol (lib_id "ao_symbols:AudioJack2") (at 93.98 125.73 0) (mirror x) (unit 1)
     (in_bom yes) (on_board no)
-    (property "Reference" "J13" (id 0) (at 89.408 125.2982 0)
+    (property "Reference" "J23" (id 0) (at 89.408 125.2982 0)
       (effects (font (size 1.27 1.27)) (justify right))
     )
@@
   (symbol (lib_id "ao_symbols:R_POT") (at 156.21 130.81 270) (unit 1)
     (in_bom yes) (on_board no)
-    (property "Reference" "RV1" (id 0) (at 156.21 125.5522 90))
+    (property "Reference" "RV5" (id 0) (at 156.21 125.5522 90))
     (property "Value" "100k" (id 1) (at 156.21 127.8636 90))
     (property "Footprint" "ao_tht:Potentiometer_Alpha_RD901F-40-00D_Single_Vertical_centered" (id 2) (at 156.21 130.81 0)
@@
   (symbol (lib_id "ao_symbols:AudioJack2") (at 95.25 158.75 180) (unit 1)
     (in_bom yes) (on_board no)
-    (property "Reference" "J15" (id 0) (at 99.822 158.3182 0)
+    (property "Reference" "J25" (id 0) (at 99.822 158.3182 0)
       (effects (font (size 1.27 1.27)) (justify right))
     )
@@
   (symbol (lib_id "power:GND1") (at 100.33 129.54 0) (mirror y) (unit 1)
     (in_bom yes) (on_board yes)
-    (property "Reference" "#PWR05" (id 0) (at 100.33 135.89 0)
+    (property "Reference" "#PWR047" (id 0) (at 100.33 135.89 0)
       (effects (font (size 1.27 1.27)) hide)
     )
@@
   (symbol (lib_id "ao_symbols:AudioJack2") (at 95.25 143.51 180) (unit 1)
     (in_bom yes) (on_board no)
-    (property "Reference" "J14" (id 0) (at 99.822 143.0782 0)
+    (property "Reference" "J24" (id 0) (at 99.822 143.0782 0)
       (effects (font (size 1.27 1.27)) (justify right))
     )
@@
     (pin "T")
   )
-  (symbol (lib_name "SW_DP3T_1") (lib_id "herovco:SW_DP3T") (at 186.69 82.55 0) (unit 1)
+  (symbol (lib_id "herovco:SW_DP3T") (at 186.69 82.55 0) (unit 1)
     (in_bom yes) (on_board yes) (fields_autoplaced)
     (property "Reference" "SW2" (id 0) (at 186.69 75.7133 0))
@@
   (symbol (lib_id "power:GND1") (at 88.9 162.56 0) (unit 1)
     (in_bom yes) (on_board yes)
-    (property "Reference" "#PWR04" (id 0) (at 88.9 168.91 0)
+    (property "Reference" "#PWR046" (id 0) (at 88.9 168.91 0)
       (effects (font (size 1.27 1.27)) hide)
     )
@@
   )
   (symbol (lib_id "ao_symbols:Board") (at 203.2 27.94 0) (unit 1)
-    (in_bom yes) (on_board yes) (fields_autoplaced)
+    (in_bom no) (on_board yes) (fields_autoplaced)
     (property "Reference" "B2" (id 0) (at 208.915 27.0315 0)
       (effects (font (size 1.27 1.27)) (justify left))

Commit message: Fix nuked footprints; update trimmer footprints
Parts:
- B2: footprint ao_tht:Board_Marker -> (none)
- GRAF4: value board -> (none); footprint sidekickvco:sidekick_daughterboard -> (none)
- H1, H2: footprint ao_tht:MountingHole_3.2mm_M3 -> (none)
- J23, J24, J25: footprint ao_tht:Jack_6.35mm_PJ_629HAN -> (none)
- R30, R31, R32, R33: footprint ao_tht:R_Axial_DIN0207_L6.3mm_D2.5mm_P10.16mm_Horizontal -> (none)
- RV5: footprint ao_tht:Potentiometer_Alpha_RD901F-40-00D_Single_Vertical_centered -> (none)
- SW1: footprint ao_tht:Rotary_Switch -> (none)
- SW2: footprint herovco:SW_CK_OS203012MU5QP1_DP3T -> (none)
Changed lines of the file:
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@@
     (property "Reference" "SW1" (id 0) (at 118.11 43.815 0))
     (property "Value" "SW_Rotary12" (id 1) (at 118.11 46.1264 0))
-    (property "Footprint" "ao_tht:Rotary_Switch" (id 2) (at 120.65 82.55 0)
+    (property "Footprint" "" (id 2) (at 120.65 82.55 0)
       (effects (font (size 1.27 1.27)) hide)
     )
@@
       (effects (font (size 1.27 1.27)) (justify left))
     )
-    (property "Footprint" "ao_tht:R_Axial_DIN0207_L6.3mm_D2.5mm_P10.16mm_Horizontal" (id 2) (at 82.042 53.34 90)
+    (property "Footprint" "" (id 2) (at 82.042 53.34 90)
       (effects (font (size 1.27 1.27)) hide)
     )
@@
       (effects (font (size 1.27 1.27)) (justify left))
     )
-    (property "Footprint" "ao_tht:R_Axial_DIN0207_L6.3mm_D2.5mm_P10.16mm_Horizontal" (id 2) (at 82.042 60.96 90)
+    (property "Footprint" "" (id 2) (at 82.042 60.96 90)
       (effects (font (size 1.27 1.27)) hide)
     )
@@
       (effects (font (size 1.27 1.27)) (justify left))
     )
-    (property "Footprint" "ao_tht:R_Axial_DIN0207_L6.3mm_D2.5mm_P10.16mm_Horizontal" (id 2) (at 82.042 68.58 90)
+    (property "Footprint" "" (id 2) (at 82.042 68.58 90)
       (effects (font (size 1.27 1.27)) hide)
     )
@@
       (effects (font (size 1.27 1.27)) (justify left))
     )
-    (property "Footprint" "ao_tht:R_Axial_DIN0207_L6.3mm_D2.5mm_P10.16mm_Horizontal" (id 2) (at 82.042 76.2 90)
+    (property "Footprint" "" (id 2) (at 82.042 76.2 90)
       (effects (font (size 1.27 1.27)) hide)
     )
@@
       (effects (font (size 1.27 1.27)) (justify left))
     )
-    (property "Value" "board" (id 1) (at 208.915 39.9666 0)
-      (effects (font (size 1.27 1.27)) (justify left))
-    )
-    (property "Footprint" "sidekickvco:sidekick_daughterboard" (id 2) (at 201.93 38.1 0)
+    (property "Value" "" (id 1) (at 208.915 39.9666 0)
+      (effects (font (size 1.27 1.27)) (justify left))
+    )
+    (property "Footprint" "" (id 2) (at 201.93 38.1 0)
       (effects (font (size 1.27 1.27)) hide)
     )
@@
       (effects (font (size 1.27 1.27)) (justify right))
     )
-    (property "Footprint" "ao_tht:Jack_6.35mm_PJ_629HAN" (id 2) (at 93.98 125.73 0)
+    (property "Footprint" "" (id 2) (at 93.98 125.73 0)
       (effects (font (size 1.27 1.27)) hide)
     )
@@
     (property "Reference" "RV5" (id 0) (at 156.21 125.5522 90))
     (property "Value" "100k" (id 1) (at 156.21 127.8636 90))
-    (property "Footprint" "ao_tht:Potentiometer_Alpha_RD901F-40-00D_Single_Vertical_centered" (id 2) (at 156.21 130.81 0)
+    (property "Footprint" "" (id 2) (at 156.21 130.81 0)
       (effects (font (size 1.27 1.27)) hide)
     )
@@
       (effects (font (size 1.27 1.27)) (justify right))
     )
-    (property "Footprint" "ao_tht:Jack_6.35mm_PJ_629HAN" (id 2) (at 95.25 158.75 0)
+    (property "Footprint" "" (id 2) (at 95.25 158.75 0)
       (effects (font (size 1.27 1.27)) hide)
     )
@@
       (effects (font (size 1.27 1.27)) (justify left))
     )
-    (property "Footprint" "ao_tht:MountingHole_3.2mm_M3" (id 2) (at 204.47 54.61 0)
+    (property "Footprint" "" (id 2) (at 204.47 54.61 0)
       (effects (font (size 1.27 1.27)) hide)
     )
@@
       (effects (font (size 1.27 1.27)) (justify right))
     )
-    (property "Footprint" "ao_tht:Jack_6.35mm_PJ_629HAN" (id 2) (at 95.25 143.51 0)
+    (property "Footprint" "" (id 2) (at 95.25 143.51 0)
       (effects (font (size 1.27 1.27)) hide)
     )
@@
     (property "Reference" "SW2" (id 0) (at 186.69 75.7133 0))
     (property "Value" "SW_DP3T" (id 1) (at 186.69 78.4884 0))
-    (property "Footprint" "herovco:SW_CK_OS203012MU5QP1_DP3T" (id 2) (at 170.815 78.105 0)
+    (property "Footprint" "" (id 2) (at 170.815 78.105 0)
       (effects (font (size 1.27 1.27)) hide)
     )
@@
       (effects (font (size 1.27 1.27)) (justify left))
     )
-    (property "Footprint" "ao_tht:MountingHole_3.2mm_M3" (id 2) (at 204.47 48.26 0)
+    (property "Footprint" "" (id 2) (at 204.47 48.26 0)
       (effects (font (size 1.27 1.27)) hide)
     )
@@
     (property "Reference" "SW2" (id 0) (at 173.99 61.7433 0))
     (property "Value" "SW_DP3T" (id 1) (at 173.99 64.5184 0))
-    (property "Footprint" "herovco:SW_CK_OS203012MU5QP1_DP3T" (id 2) (at 158.115 64.135 0)
+    (property "Footprint" "" (id 2) (at 158.115 64.135 0)
       (effects (font (size 1.27 1.27)) hide)
     )
@@
       (effects (font (size 1.27 1.27)) (justify left))
     )
-    (property "Footprint" "ao_tht:Board_Marker" (id 2) (at 203.2 27.94 0)
-      (effects (font (size 1.27 1.27)) hide)
-    )
+    (property "Footprint" "" (id 2) (at 203.2 27.94 0)
+      (effects (font (size 1.27 1.27)) hide)
+    )
