File: Hardware/PCB/sidekickvco/panel.kicad_sch (KiCad schematic)
At the start: 14 parts, among them J23 AudioJack2, J24 AudioJack2, J25 AudioJack2, SW1 SW_Rotary12, SW2 SW_DP3T

Commit message: Post prototype updates
Parts:
- B2: footprint (none) -> ao_tht:Board_Marker
- GRAF4: value (none) -> board; footprint (none) -> sidekickvco:sidekick_daughterboard
- H1, H2: footprint (none) -> ao_tht:MountingHole_3.2mm_M3
- RV5: SKU (none) -> A-5606 or A-1984
- SW2: footprint (none) -> sidekickvco:SW_CK_OS203012MU5QP1_DP3T
Changed lines of the file:
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@@
       (effects (font (size 1.27 1.27)) (justify left))
     )
-    (property "Value" "" (id 1) (at 208.915 39.9666 0)
-      (effects (font (size 1.27 1.27)) (justify left))
-    )
-    (property "Footprint" "" (id 2) (at 201.93 38.1 0)
+    (property "Value" "board" (id 1) (at 208.915 39.9666 0)
+      (effects (font (size 1.27 1.27)) (justify left))
+    )
+    (property "Footprint" "sidekickvco:sidekick_daughterboard" (id 2) (at 201.93 38.1 0)
       (effects (font (size 1.27 1.27)) hide)
     )
@@
       (effects (font (size 1.27 1.27)) hide)
     )
+    (property "Description" "1/4\" audio jack, vertical" (id 6) (at 93.98 125.73 0)
+      (effects (font (size 1.27 1.27)) hide)
+    )
     (pin "S")
     (pin "T")
@@
       (effects (font (size 1.27 1.27)) hide)
     )
+    (property "Description" "Panel mount linear potentiometer" (id 5) (at 156.21 130.81 0)
+      (effects (font (size 1.27 1.27)) hide)
+    )
+    (property "SKU" "A-5606 or A-1984" (id 6) (at 156.21 130.81 0)
+      (effects (font (size 1.27 1.27)) hide)
+    )
     (pin "1")
     (pin "2")
@@
     )
     (property "SKU" "A-1121" (id 5) (at 95.25 158.75 0)
+      (effects (font (size 1.27 1.27)) hide)
+    )
+    (property "Description" "1/4\" audio jack, vertical" (id 6) (at 95.25 158.75 0)
       (effects (font (size 1.27 1.27)) hide)
     )
@@
       (effects (font (size 1.27 1.27)) (justify left))
     )
-    (property "Footprint" "" (id 2) (at 204.47 54.61 0)
+    (property "Footprint" "ao_tht:MountingHole_3.2mm_M3" (id 2) (at 204.47 54.61 0)
       (effects (font (size 1.27 1.27)) hide)
     )
@@
     )
     (property "SKU" "A-1121" (id 5) (at 95.25 143.51 0)
+      (effects (font (size 1.27 1.27)) hide)
+    )
+    (property "Description" "1/4\" audio jack, vertical" (id 6) (at 95.25 143.51 0)
       (effects (font (size 1.27 1.27)) hide)
     )
@@
     (property "Reference" "SW2" (id 0) (at 186.69 75.7133 0))
     (property "Value" "SW_DP3T" (id 1) (at 186.69 78.4884 0))
-    (property "Footprint" "" (id 2) (at 170.815 78.105 0)
+    (property "Footprint" "sidekickvco:SW_CK_OS203012MU5QP1_DP3T" (id 2) (at 170.815 78.105 0)
       (effects (font (size 1.27 1.27)) hide)
     )
@@
       (effects (font (size 1.27 1.27)) (justify left))
     )
-    (property "Footprint" "" (id 2) (at 204.47 48.26 0)
+    (property "Footprint" "ao_tht:MountingHole_3.2mm_M3" (id 2) (at 204.47 48.26 0)
       (effects (font (size 1.27 1.27)) hide)
     )
@@
     (property "Reference" "SW2" (id 0) (at 173.99 61.7433 0))
     (property "Value" "SW_DP3T" (id 1) (at 173.99 64.5184 0))
-    (property "Footprint" "" (id 2) (at 158.115 64.135 0)
+    (property "Footprint" "sidekickvco:SW_CK_OS203012MU5QP1_DP3T" (id 2) (at 158.115 64.135 0)
       (effects (font (size 1.27 1.27)) hide)
     )
@@
       (effects (font (size 1.27 1.27)) (justify left))
     )
-    (property "Footprint" "" (id 2) (at 203.2 27.94 0)
-      (effects (font (size 1.27 1.27)) hide)
-    )
+    (property "Footprint" "ao_tht:Board_Marker" (id 2) (at 203.2 27.94 0)
+      (effects (font (size 1.27 1.27)) hide)
+    )
