File: Hardware/PCB/sidekickvco/sidekickvco_outputs.kicad_sch (KiCad schematic)
At the start: 36 parts, among them Q1 2N3904, Q2 2N3904, U7 TL074

Commit message: Initial version of circuit and layout
Connections:
- net +12V_1 renamed +12V
- net -12V_1 renamed -12V
- net GND1 renamed GND
- net PULSE_OUT_S renamed PULSE_OUT
- net SAW_OUT_S renamed SAW_OUT
- net TRIANGLE_OUT_S renamed TRIANGLE_OUT
Other:
- note removed: "SINE TRIMMERS"

Commit message: 5 mm pitch for 330 pF
Parts:
- C18, C19: footprint ao_tht:C_Disc_D3.0mm_W1.6mm_P2.50mm -> ao_tht:C_Disc_D5.0mm_W2.5mm_P5.00mm
Changed lines of the file:
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@@
     (property "Reference" "C18" (id 0) (at 222.25 86.3092 90))
     (property "Value" "330pF" (id 1) (at 222.25 88.6206 90))
-    (property "Footprint" "ao_tht:C_Disc_D3.0mm_W1.6mm_P2.50mm" (id 2) (at 218.44 93.6752 0)
+    (property "Footprint" "ao_tht:C_Disc_D5.0mm_W2.5mm_P5.00mm" (id 2) (at 218.44 93.6752 0)
       (effects (font (size 1.27 1.27)) hide)
     )
@@
     (property "Reference" "C19" (id 0) (at 222.25 120.5992 90))
     (property "Value" "330pF" (id 1) (at 222.25 122.9106 90))
-    (property "Footprint" "ao_tht:C_Disc_D3.0mm_W1.6mm_P2.50mm" (id 2) (at 218.44 127.9652 0)
+    (property "Footprint" "ao_tht:C_Disc_D5.0mm_W2.5mm_P5.00mm" (id 2) (at 218.44 127.9652 0)
       (effects (font (size 1.27 1.27)) hide)
     )

Commit message: Pre prototype revisions, README revision
Parts:
- renumbered C16 to C15, C17 to C16, C18 to C17, C19 to C18, R42 to R34, R43 to R35, R44 to R36, R45 to R37, R46 to R38, R47 to R39, R48 to R40, R49 to R41, R50 to R42, R51 to R43, R52 to R44, R53 to R45, R54 to R46, R55 to R47, R56 to R48, R57 to R49, R58 to R50, R59 to R51, R60 to R52, R61 to R53, R62 to R54, R63 to R55, R64 to R56, R65 to R57, R66 to R58, R67 to R59, RV10 to RV6, RV11 to RV7, RV12 to RV8, U7 to U6

Commit message: Fix nuked footprints; update trimmer footprints
Parts:
- C15, C16: footprint ao_tht:C_Disc_D3.0mm_W1.6mm_P2.50mm -> (none)
- C17, C18: footprint ao_tht:C_Disc_D5.0mm_W2.5mm_P5.00mm -> (none)
- Q1, Q2: footprint ao_tht:TO-92_Inline_Wide -> (none)
- R34, R35, R36, R37, R38, R39, R40, R41, R42, R43, R44, R45, R46, R47, R48, R49, R50, R51, R52, R53, R54, R55, R56, R57, R58, R59: footprint ao_tht:R_Axial_DIN0207_L6.3mm_D2.5mm_P10.16mm_Horizontal -> (none)
- RV6, RV7, RV8: footprint ao_tht:Potentiometer_Bourns_3296W_Vertical_screw_centered -> (none)
- U6: footprint ao_tht:DIP-14_W7.62mm_Socket_LongPads -> (none)

Commit message: Post prototype updates
Parts:
- C15, C16: footprint (none) -> ao_tht:C_Disc_D3.0mm_W1.6mm_P2.50mm
- C17, C18: footprint (none) -> ao_tht:C_Disc_D5.0mm_W2.5mm_P5.00mm
- Q1, Q2: footprint (none) -> ao_tht:TO-92_Inline_Wide
- R34, R35, R36, R37, R38, R39, R40, R41, R42, R43, R44, R45, R46, R47, R48, R49, R50, R51, R52, R53, R54, R55, R56, R57, R58, R59: footprint (none) -> ao_tht:R_Axial_DIN0207_L6.3mm_D2.5mm_P10.16mm_Horizontal
- RV6, RV7: footprint (none) -> ao_tht:Potentiometer_Bourns_3296W_Vertical_screw_centered; SKU (none) -> A-598
- RV8: footprint (none) -> ao_tht:Potentiometer_Bourns_3296W_Vertical_screw_centered; SKU (none) -> A-597
- U6: footprint (none) -> ao_tht:DIP-14_W7.62mm_Socket_LongPads
