File: Hardware/PCB/sidekickvco/Separate PCBs/sidekickvco_b2.kicad_pcb (KiCad board)
At the start: 2 copper layers, 25 x 24 mm, 8 parts, among them J14 Wire pad, J15 Wire pad, J16 Wire pad, J17 Wire pad, SW2 SW_DP3T

Commit message: Post prototype updates
Parts:
- SW2: footprint herovco:SW_CK_OS203012MU5QP1_DP3T -> sidekickvco:SW_CK_OS203012MU5QP1_DP3T
