File: Hardware/PCB/sidekickvco/Separate PCBs/sidekickvco_b1.kicad_pcb (KiCad board)
At the start: 2 copper layers, 81 x 163 mm, 113 parts, among them J1 Conn_02x04_Odd_Even, J18 AudioJack2, J19 AudioJack2, J2 3_pin_Molex_header, J20 Synth_power_2x5, J21 AudioJack2, J22 AudioJack2, J3 3_pin_Molex_header, J4 4_pin_Molex_header, J5 2_pin_Molex_header, J6 2_pin_Molex_header, J7 2_pin_Molex_header, Q1 2N3904, Q2 2N3904, U1 TL072, U2 AS3340A, U3 LM4040BIZ-5, U4 LM4040BIZ-5, U5 L79L05_TO92, U6 TL074

Commit message: Post prototype updates
Parts:
- removed B1: Board, ao_tht:Board_Marker
- removed J18, J19, J21, J22: AudioJack2, ao_tht:Jack_6.35mm_TE-CK-6.35-29B_Horizontal
- removed RV1, RV2, RV3, RV4: 10k, Potentiometer_THT:Potentiometer_Bourns_3296P_Horizontal
- moved R23 69.0 mm to (148.9, 29.3)
- moved U3 18.3 mm to (128.6, 23.3)
- moved C1 9.53 mm to (132.3, 62.3)
- moved C11 9.53 mm to (175.6, 81.3)
- moved C13 9.53 mm to (143.7, 142.3)
- moved C14 9.53 mm to (137.3, 142.3)
- moved C15 9.53 mm to (148.8, 125.8)
- moved C16 9.53 mm to (128.5, 125.8)
- moved C3 9.53 mm to (138.7, 44.5)
- moved C6 9.53 mm to (148.8, 54.7)
- moved D1 9.53 mm to (142.5, 77.5)
- moved GRAF2 9.53 mm to (149.9, 170.5)
- moved GRAF3 9.53 mm to (182.4, 22.2)
- moved J7 9.53 mm to (157.7, 160.1)
- moved R12 9.53 mm to (165.4, 77.5)
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Routing:
- net Board_0-+5V_REF: track 188.2 -> 110.0 mm
- net Board_0-Net-(R25-Pad1): track 21.7 -> 31.8 mm
- net Board_0-+12V: track 237.0 -> 242.2 mm
- net Board_0-/Main PCB/LINK_IN_PW: track 63.7 -> 59.2 mm
- net Board_0-PWMIN: track 77.8 -> 73.9 mm
- net Board_0-Net-(R28-Pad1): track 45.0 -> 42.2 mm
- net Board_0-Net-(C4-Pad1): track 19.5 -> 21.9 mm
- net Board_0-/Main PCB/LIN_FM_IN: track 19.4 -> 17.8 mm
- net Board_0--5V_REF: track 49.0 -> 47.5 mm
- net Board_0-/Main PCB/HI_FREQ_TRACK: track 19.0 -> 20.0 mm
- net Board_0-PWM_IN: track 63.2 -> 64.2 mm
- net Board_0-Net-(R4-Pad2): track 29.5 -> 30.5 mm
- net Board_0-HFT: track 50.8 -> 51.8 mm
- net Board_0--5V: track 97.2 -> 98.2 mm
- net Board_0-/Main PCB/CENTER_FREQ: track 14.9 -> 15.9 mm
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Other:
- board text added: "Match R8-R10 Match R1-R2 with octave switch"
- board text added: "Match with R8/10"
- board text added: "Match with R9"
- board text added: "Match with oct switch"

Commit message: Fix lin FM input, add howitworks
Parts:
- removed R7: 100k, ao_tht:R_Axial_DIN0207_L6.3mm_D2.5mm_P10.16mm_Horizontal
Connections:
- C4 pad 2: Board_0-Net-(C4-Pad2) -> Board_0-/Main PCB/LIN_FM_IN
- C5 pad 2: Board_0-Net-(C5-Pad2) -> Board_0-/Main PCB/LINK_IN_FM
- R6 pad 1: Board_0-Net-(C4-Pad2) -> Board_0-/Main PCB/LIN_FM_IN
- R6 pad 2: Board_0-/Main PCB/LIN_FM_IN -> Board_0-GND
Routing:
- net Board_0-/Main PCB/LINK_IN_FM: track 31.3 -> 43.5 mm, vias 0 -> 1
- net Board_0-Net-(C5-Pad2): track 11.0 -> 0.00 mm
- net Board_0-Net-(C4-Pad2): track 6.74 -> 0.00 mm
- net Board_0-/Main PCB/LIN_FM_IN: track 17.8 -> 14.4 mm

Commit message: Restore resistor
Parts:
- added R7: 100k, ao_tht:R_Axial_DIN0207_L6.3mm_D2.5mm_P10.16mm_Horizontal, F.Cu at (129.9, 54.7)
Routing:
- net Board_0-/Main PCB/LINK_IN_FM: vias 1 -> 0

Commit message: New b1 Gerbers
Parts:
- added B1: Board, ao_tht:Board_Marker, F.Cu at (144.6, 21.0)
- added J18: AudioJack2, ao_tht:Jack_6.35mm_TE-CK-6.35-29B_Horizontal, F.Cu at (169.5, 113.9)
- added J19: AudioJack2, ao_tht:Jack_6.35mm_TE-CK-6.35-29B_Horizontal, F.Cu at (169.5, 88.9)
- added J21: AudioJack2, ao_tht:Jack_6.35mm_TE-CK-6.35-29B_Horizontal, F.Cu at (169.5, 138.9)
- added J22: AudioJack2, ao_tht:Jack_6.35mm_TE-CK-6.35-29B_Horizontal, F.Cu at (169.5, 163.9)
- added RV1: 10k, ao_tht:Potentiometer_Bourns_3296P_Horizontal, F.Cu at (182.3, 57.0)
- added RV2: 10k, ao_tht:Potentiometer_Bourns_3296P_Horizontal, F.Cu at (182.3, 81.0)
- added RV3: 10k, ao_tht:Potentiometer_Bourns_3296P_Horizontal, F.Cu at (182.3, 45.0)
- added RV4: 50k, ao_tht:Potentiometer_Bourns_3296P_Horizontal, F.Cu at (182.3, 69.0)
- moved C1 4.89 mm to (128.1, 64.8)
- moved C11 4.89 mm to (171.4, 83.8)
- moved C13 4.89 mm to (139.5, 144.8)
- moved C14 4.89 mm to (133.1, 144.8)
- moved C15 4.89 mm to (144.6, 128.3)
- moved C16 4.89 mm to (124.3, 128.3)
- moved C3 4.89 mm to (134.5, 47.0)
- moved C4 4.89 mm to (156.1, 94.0)
- moved C6 4.89 mm to (144.6, 57.2)
- moved D1 4.89 mm to (138.3, 80.0)
- moved GRAF2 4.89 mm to (145.7, 173.0)
- moved GRAF3 4.89 mm to (178.2, 24.7)
- moved J7 4.89 mm to (153.5, 162.6)
- moved R12 4.89 mm to (161.2, 80.0)
- moved R14 4.89 mm to (161.2, 52.1)
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